File: pcb/benchpod/LogicAnalyzer.kicad_sch (KiCad schematic)
At the start: 54 parts, among them U18 SN74LVC2G66DCUR, U19 SN74LVC2G66DCUR, U20 SN74LVC2G66DCUR, U21 SN74LVC2G66DCUR, U22 SRV05-4.TCT, U23 SRV05-4.TCT, U25 SRV05-4.TCT, U34 SRV05-4.TCT, U54 TCA9554PWR

Commit message: 1V8/3V3 pull-ups / pull-down fixes
Connections:
- net +3V3: no longer R38.1, R39.1, R50.2, R51.2, R58.1, R62.2
- new net LA_VCCIO: R38.1, R39.1, R50.2, R51.2, R58.1, R62.2
