File: pcb/benchpod/LogicAnalyzer.kicad_sch (KiCad schematic)
At the start: 54 parts, among them U18 SN74LVC2G66DCUR, U19 SN74LVC2G66DCUR, U20 SN74LVC2G66DCUR, U21 SN74LVC2G66DCUR, U22 SRV05-4.TCT, U23 SRV05-4.TCT, U25 SRV05-4.TCT, U34 SRV05-4.TCT, U54 TCA9554PWR

Commit message: analog v3r2: no extra BOM lines from the 0.1 % swaps and cap shrinks
JLC standard assembly charges per unique BOM line, so only keep changes
that replace a whole line:
- Revert 4.7 uF C2 C3 C5 C220 and 22 uF C16 C108 C154 C157 to 0805 (the
  other 4.7 uF/22 uF stay 0805, so the shrink split a line), and 5.1 pF C207
  C208 to the 0603 C2297586 (C140 needs it; 29 in stock = 9 boards).
- Move the remaining 1k (R21 R22 R164 R175), 1.5k (R15) and 2.2k (R58 R62)
  to the same 0.1 % parts as the precision ones, so their old lines go.

BOM: 122 -> 124 unique lines (0.1 % 10k for R109 R110 R111 R123, tantalum
C142). Netlist connectivity unchanged.

Co-Authored-By: Claude Opus 5.5 <noreply@anthropic.com>
Parts:
- R58, R62: LCSC C25879 -> C326602
Changed lines of the file:
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@@
 			)
 		)
-		(property "LCSC" "C25879"
+		(property "LCSC" "C326602"
 			(at 106.68 124.46 0)
 			(hide yes)
@@
 			)
 		)
-		(property "LCSC" "C25879"
+		(property "LCSC" "C326602"
 			(at 147.32 140.97 0)
 			(hide yes)
