File: pcb/benchpod/power.kicad_sch (KiCad schematic)
At the start: 64 parts, among them J4 Screw_Terminal_01x02, J5 Screw_Terminal_01x02, J6 Screw_Terminal_01x02, U26 TPS259470ARPWR, U27 TPS259470ARPWR, U28 USBLC6-2SC6, U29 INA219AxDCN, U30 TPS82130SILR, U31 AP2112K-1.2, U32 AP2112K-2.5TRG1, U33 INA219AxDCN

Commit message: v2.0.0
Parts:
- removed C91, C92: 22u, Capacitor_SMD:C_0603_1608Metric, symbol Device:C
- removed C93: 10u, Capacitor_SMD:C_0603_1608Metric, symbol Device:C
- removed D7: D_TVS, lcsc:SOD-523_L1.2-W0.8-LS1.6-RD, symbol Device:D_TVS
- removed D8, D9: Green LED, lcsc:LED0805-RD, symbol Device:LED
- removed R75, R76: 5.1k, Resistor_SMD:R_0402_1005Metric, symbol Device:R
- removed R81, R82: 1k, Resistor_SMD:R_0402_1005Metric, symbol Device:R
- removed U28: USBLC6-2SC6, lcsc:SOT-23-6_L2.9-W1.6-P0.95-LS2.8-BL, symbol Power_Protection:USBLC6-2SC6
- removed U29, U33: INA219AxDCN, lcsc:SOT-23-8_L3.0-W1.7-P0.65-LS2.8-BR, symbol Sensor_Energy:INA219AxDCN
- removed USBC1: TYPE-C-31-M-12, lcsc:USB-C_SMD-TYPE-C-31-M-12_1, symbol lcsc_lib:TYPE-C-31-M-12
- added C123: 10u, Capacitor_SMD:C_0603_1608Metric, symbol Device:C
- added C125, C163, C216, C221, C223: 100n, Capacitor_SMD:C_0402_1005Metric, symbol Device:C
- added C217, C222, C240: 1u, Capacitor_SMD:C_0402_1005Metric, symbol Device:C
- added D5: SMAJ22A_C41376403, lcsc:SMA_L4.3-W2.6-LS5.0-RD, symbol lcsc_lib:SMAJ22A_C41376403
- added R137: 10k, Resistor_SMD:R_0402_1005Metric, symbol Device:R
- added U29, U33: INA238AIDGSR, lcsc:VSSOP-10_L3.0-W3.0-P0.50-LS4.9-BL, symbol lcsc_lib:INA238AIDGSR
- added U52: AP2112K-1.8TRG1, lcsc:SOT-25_L3.0-W1.6-P0.95-LS2.8-BL, symbol lcsc_lib:AP2112K-1.8TRG1
- added U56: TCA9554PWR, lcsc:TSSOP-16_L5.0-W4.4-P0.65-LS6.4-TL, symbol lcsc_lib:TCA9554PWR
- C101, C109, C112, C113, C114, C116, C118, C94, C96, C98: footprint Capacitor_SMD:C_0603_1608Metric -> Capacitor_SMD:C_0402_1005Metric; LCSC C14663 -> C307331
- C107, C110, C111, C115, C117: footprint Capacitor_SMD:C_0603_1608Metric -> Capacitor_SMD:C_0402_1005Metric; LCSC C15849 -> C1518208
Connections:
- net +3V3: now also C123.2, C125.2, C216.1, C217.2, C221.2, C240.2, R137.1, U29.6 (VS), U33.1 (A1), U33.6 (VS), U52.1 (VIN), U52.3 (EN), U56.16 (VCC), U56.2 (A1)
- net 2V5: now also C163.2
- net EFUSE1_ENABLE: now also U56.12 (P7)
- net EFUSE1_FLT: now also U56.10 (P5)
- net EFUSE1_V: now also U56.11 (P6)
- net EFUSE2_ENABLE: now also U56.4 (PO)
- net EFUSE2_FLT: now also U56.6 (P2)
- net EFUSE2_V: now also U56.5 (P1)
- net GND: now also C123.1, C125.1, C163.1, C216.2, C217.1, C221.1, C222.1, C223.1, C240.1, D5.2 (A), U29.1 (A1), U29.2 (A0), U29.7 (GND), U33.2 (A0), U33.7 (GND), U52.2 (GND), U56.1 (AO), U56.3 (A2), U56.8 (GND)
- net INA_IN_M1: now also U29.8 (VBUS), U29.9 (IN-)
- net INA_IN_M2: now also U33.8 (VBUS), U33.9 (IN-)
- net INA_IN_P1: now also U29.10 (IN+)
- net INA_IN_P2: now also U33.10 (IN+)
- net INA_SCL: now also U29.5 (SCL), U33.5 (SCL)
- net INA_SDA: now also U29.4 (SDA), U33.4 (SDA)
- net at C96.2, C97.1, J4.1 (Pin_1)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: now also D5.1 (C)
- new net +1V8: C222.2, C223.2, U52.5 (VOUT)
- new net EFUSE_INT: R137.2, U56.13 (#INT)
- new net INA1_ALERT: U29.3 (ALERT), U56.9 (P4)
- new net INA2_ALERT: U33.3 (ALERT), U56.7 (P3)
- new net SCL: U56.14 (SCL)
- new net SDA: U56.15 (SDA)
- no-connect marks 4 -> 3
Other:
- note added: "Address 0x22"
- note added: "C0G"
- note added: "GPIO Control"
- note added: "Power (5V to +3V3, 1V2, 1V8, 2V5)"
- note removed: "Address 0x41"
- note removed: "Power (5V to +3V3, 1V2, 2V5)"
- note removed: "USB Protection"
- note removed: "USB-C"
- moved on the sheet: C106, C107, C108, C109, C110, C111, C113, C114, C115, C116, C117, C119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
