File: pcb/benchpod/power.kicad_sch (KiCad schematic)
At the start: 70 parts, among them J4 Screw_Terminal_01x02, J5 Screw_Terminal_01x02, J6 Screw_Terminal_01x02, U26 TPS259470ARPWR, U27 TPS259470ARPWR, U29 INA226, U30 TPS82130SILR, U31 AP2112K-1.2, U32 AP2112K-2.5TRG1, U33 INA226, U52 AP2112K-1.8TRG1, U56 TCA9554PWR

Commit message: analog v3r2: lead-free diodes and SMA, 0.1 % gain resistors, tantalum ADC reference cap
RoHS/REACH (no exemption claimed in the LCSC test reports):
- SS34 D3 D9 D15 D16 -> FOSAN SS34 C3014011
- SMAJ20A D5 -> FOSAN SMAJ20A C5353170
- SMAJ36CA D6 D7 D8 D10 -> FOSAN SMAJ36CA C5353135
- SMA RF1-RF4 -> HCTL HC-SMA-KWE-14.5H-D002-01 C41410437 (same footprint,
  5.08 vs 5.10 mm pin square)
- 11.8k R127 R129 R132 R133 (RALEC, lead glass) -> YAGEO 0.1 % C852496

0.1 % 25 ppm thin film, to cut the pod-to-pod offset and gain spread:
- THS4551 gain R92 R93 (1k C852624), R94 R102 (1.5k C281775): the 1 %
  mismatch turned VOCM into an ADC offset of about +-66 mV between pods
- +-12 V difference amps R126 R128 R130 R131 (2k C852711)
- VMID divider R110 R111, 3.3 V/5 V gains R108 (C861300), R109 R123
  (10k C190095), R122 (2.2k C326602)

C142 (MCP33131 VREF) 10 uF 0603 ceramic -> 10 uF tantalum case A C7171,
pin 1 (+) on AREF_4V096. Footprint change: needs a PCB update.

Netlist connectivity unchanged (pin-to-net diff identical), ERC unchanged.

Co-Authored-By: Claude Opus 5.5 <noreply@anthropic.com>
Parts:
- D5: LCSC C41376408 -> C5353170; MPN (none) -> SMAJ20A; Manufacturer R+O(宏嘉诚) -> FOSAN
Changed lines of the file:
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@@
 			)
 		)
-		(property "LCSC" "C41376408"
+		(property "LCSC" "C5353170"
 			(at 43.18 187.96 0)
 			(hide yes)
@@
 			)
 		)
-		(property "Manufacturer" "R+O(宏嘉诚)"
+		(property "Manufacturer" "FOSAN"
 			(at 43.18 187.96 0)
 			(hide yes)
+			(show_name no)
+			(do_not_autoplace no)
+			(effects
+				(font
+					(size 1.27 1.27)
+				)
+			)
+		)
+		(property "MPN" "SMAJ20A"
+			(at 43.18 187.96 0)
+			(hide yes)
