File: pcb/benchpod/power.kicad_sch (KiCad schematic)
At the start: 70 parts, among them J4 Screw_Terminal_01x02, J5 Screw_Terminal_01x02, J6 Screw_Terminal_01x02, U26 TPS259470ARPWR, U27 TPS259470ARPWR, U29 INA226, U30 TPS82130SILR, U31 AP2112K-1.2, U32 AP2112K-2.5TRG1, U33 INA226, U52 AP2112K-1.8TRG1, U56 TCA9554PWR

Commit message: analog v3r2: smaller capacitor packages (same rating and dielectric)
To 0402: 3.3 nF C99 C102 C119 C226 (C26404), 8.2 pF C0G C29 C30 C50 C51
(C1579), 5.1 pF high-Q C207 C208 (C237535; the old C2297586 had 29 in stock).
To 0603: 4.7 uF C2 C3 C5 C220 (C69335), 22 uF C16 C108 C154 C157 (C2762594),
220 nF C189 (C64705), 2.2 uF X7R VCAP C218 C219 (C415535, from 1206).

Kept: C150/C153 (4.7 uF on the ~5 V charge-pump rails, DC-bias derating),
C140 (sees up to 58 V at TVS clamp), all 10 uF and the 22 uF on >5 V rails.
Footprint changes: needs a PCB update. Netlist connectivity unchanged.

Co-Authored-By: Claude Opus 5.5 <noreply@anthropic.com>
Parts:
- C102, C119, C99: footprint Capacitor_SMD:C_0603_1608Metric -> Capacitor_SMD:C_0402_1005Metric; LCSC C1613 -> C26404
- C108: footprint Capacitor_SMD:C_0805_2012Metric -> Capacitor_SMD:C_0603_1608Metric; LCSC C45783 -> C2762594; MPN CL21B105KBFNNNE -> CL10A226MO7JZNC
Changed lines of the file:
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@@
 			)
 		)
-		(property "Footprint" "Capacitor_SMD:C_0603_1608Metric"
+		(property "Footprint" "Capacitor_SMD:C_0402_1005Metric"
 			(at 91.1352 83.82 0)
 			(hide yes)
@@
 			)
 		)
-		(property "LCSC" "C1613"
+		(property "LCSC" "C26404"
 			(at 90.17 80.01 0)
 			(hide yes)
@@
 			)
 		)
-		(property "Footprint" "Capacitor_SMD:C_0805_2012Metric"
+		(property "Footprint" "Capacitor_SMD:C_0603_1608Metric"
 			(at 192.0748 44.45 0)
 			(hide yes)
@@
 			)
 		)
-		(property "MPN" "CL21B105KBFNNNE"
+		(property "MPN" "CL10A226MO7JZNC"
 			(at 193.04 48.26 0)
 			(hide yes)
@@
 			)
 		)
-		(property "LCSC" "C45783"
+		(property "LCSC" "C2762594"
 			(at 193.04 48.26 0)
 			(hide yes)
@@
 			)
 		)
-		(property "Footprint" "Capacitor_SMD:C_0603_1608Metric"
+		(property "Footprint" "Capacitor_SMD:C_0402_1005Metric"
 			(at 98.7552 135.89 0)
 			(hide yes)
@@
 			)
 		)
-		(property "LCSC" "C1613"
+		(property "LCSC" "C26404"
 			(at 97.79 132.08 0)
 			(hide yes)
@@
 			)
 		)
-		(property "Footprint" "Capacitor_SMD:C_0603_1608Metric"
+		(property "Footprint" "Capacitor_SMD:C_0402_1005Metric"
 			(at 261.3152 31.75 0)
 			(hide yes)
@@
 			)
 		)
-		(property "LCSC" "C1613"
+		(property "LCSC" "C26404"
 			(at 260.35 27.94 0)
 			(hide yes)

Commit message: analog v3r2: no extra BOM lines from the 0.1 % swaps and cap shrinks
JLC standard assembly charges per unique BOM line, so only keep changes
that replace a whole line:
- Revert 4.7 uF C2 C3 C5 C220 and 22 uF C16 C108 C154 C157 to 0805 (the
  other 4.7 uF/22 uF stay 0805, so the shrink split a line), and 5.1 pF C207
  C208 to the 0603 C2297586 (C140 needs it; 29 in stock = 9 boards).
- Move the remaining 1k (R21 R22 R164 R175), 1.5k (R15) and 2.2k (R58 R62)
  to the same 0.1 % parts as the precision ones, so their old lines go.

BOM: 122 -> 124 unique lines (0.1 % 10k for R109 R110 R111 R123, tantalum
C142). Netlist connectivity unchanged.

Co-Authored-By: Claude Opus 5.5 <noreply@anthropic.com>
Parts:
- C108: footprint Capacitor_SMD:C_0603_1608Metric -> Capacitor_SMD:C_0805_2012Metric; LCSC C2762594 -> C45783; MPN CL10A226MO7JZNC -> CL21B105KBFNNNE
Changed lines of the file:
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@@
 			)
 		)
-		(property "Footprint" "Capacitor_SMD:C_0603_1608Metric"
+		(property "Footprint" "Capacitor_SMD:C_0805_2012Metric"
 			(at 192.0748 44.45 0)
 			(hide yes)
@@
 			)
 		)
-		(property "MPN" "CL10A226MO7JZNC"
+		(property "MPN" "CL21B105KBFNNNE"
 			(at 193.04 48.26 0)
 			(hide yes)
@@
 			)
 		)
-		(property "LCSC" "C2762594"
+		(property "LCSC" "C45783"
 			(at 193.04 48.26 0)
 			(hide yes)
