File: pcb/benchpod/vbench-pod.kicad_sch (KiCad schematic)
At the start: 104 parts, among them J1 Conn_02x10_Odd_Even, J2 Conn_02x10_Odd_Even, J3 Conn_02x10_Odd_Even, SW1 TS-1088-AR02016, SW2 TS-1088-AR02016, U1 ICE40UP5K-SG48ITR, U10 RP2350B_C42415655, U2 W25Q64JVSSIQ, U3 SN65HVD230QDR, U4 ESP32-C3-MINI-1-N4, U5 W25Q64JVSSIQ, U6 SN74LVC2G66DCTR, U7 APS6404L-3SQR-SN_C5333729, U8 SN74LVC2G66DCTR, U9 SN74LVC2G66DCTR, Y1 ABM8-272-T3

Commit message: v2.0.0
Parts:
- removed C125, C28, C29, C31, C35: 100n, Capacitor_SMD:C_0603_1608Metric, symbol Device:C
- removed C30: 4.7u, Capacitor_SMD:C_0603_1608Metric, symbol Device:C
- removed D1: Green LED, lcsc:LED0805-RD, symbol Device:LED
- removed D2: Yellow LED, lcsc:LED0805-RD, symbol Device:LED
- removed D3: Red LED, lcsc:LED0805-RD, symbol Device:LED
- removed D4: PESD2CAN,215, lcsc:SOT-23-3_L2.9-W1.3-P1.90-LS2.4-BR, symbol lcsc_lib:PESD2CAN,215
- removed J2, J3: Conn_02x10_Odd_Even, lcsc:HDR-TH_20P-P2.54-V-M-R2-C10-S2.54, symbol Connector_Generic:Conn_02x10_Odd_Even
- removed L1: 3.3u, lcsc:IND-SMD_L2.0-W1.6_AOTA-B201610S3R3-101-T, symbol Device:L
- removed R14, R20: 0, Resistor_SMD:R_0402_1005Metric, symbol Device:R
- removed R15, R7: 10k, Resistor_SMD:R_0402_1005Metric, symbol Device:R
- removed R19: 1k, Resistor_SMD:R_0402_1005Metric, symbol Device:R
- removed R23, R24: 27, Resistor_SMD:R_0402_1005Metric, symbol Device:R
- removed R25: 33, Resistor_SMD:R_0402_1005Metric, symbol Device:R
- removed TP1, TP2, TP4, TP5, TP6: TestPoint, TestPoint:TestPoint_Pad_2.0x2.0mm, symbol Connector:TestPoint
- removed U10: RP2350B_C42415655, lcsc:QFN-80_L10.0-W10.0-P0.40-TL-EP3.4, symbol lcsc_lib:RP2350B_C42415655
- removed U3: SN65HVD230QDR, lcsc:SOIC-8_L5.0-W4.0-P1.27-LS6.0-BL, symbol lcsc_lib:SN65HVD230QDR
- removed U5: W25Q64JVSSIQ, lcsc:SOIC-8_L5.3-W5.3-P1.27-LS8.0-BL, symbol edward_lib:W25Q64JVSSIQ
- removed U6, U8, U9: SN74LVC2G66DCTR, lcsc:SM-8_L3.0-W2.8-P0.65-LS4.0-BR, symbol lcsc_lib:SN74LVC2G66DCTR
- removed Y1: ABM8-272-T3, lcsc:CRYSTAL-SMD_4P-L3.2-W2.5-BL, symbol Device:Crystal_GND24
- added C121, C43, C48, C52, C54, C59, C60: 100n, Capacitor_SMD:C_0402_1005Metric, symbol Device:C
- added C122: 10u, Capacitor_SMD:C_0603_1608Metric, symbol Device:C
- added C218, C219: 2.2u, Capacitor_SMD:C_1206_3216Metric, symbol Device:C
- added C220: 4.7u, Capacitor_SMD:C_1206_3216Metric, symbol Device:C
- added C50, C51: 8.2p, Capacitor_SMD:C_0603_1608Metric, symbol Device:C
- added C53, C55: 1u, Capacitor_SMD:C_0402_1005Metric, symbol Device:C
- added FB2: FerriteBead, lcsc:L0603, symbol Device:FerriteBead
- added H1, H2, H3: HC-PZ127-7.2L-2X5PZ, lcsc:HDR-TH_HC-PZ127-7.2L-2X5PZ, symbol lcsc_lib:HC-PZ127-7.2L-2X5PZ
- added H10, H11, H12, H14: MountingHole, MountingHole:MountingHole_2.7mm_M2.5, symbol Mechanical:MountingHole
- added LED1: S4-3528RGBTA-A, lcsc:LED-SMD_4P-L3.2-W2.8-LS3.5-TL-1, symbol lcsc_lib:S4-3528RGBTA-A
- added R138, R33, R34, R35, R89: 10k, Resistor_SMD:R_0402_1005Metric, symbol Device:R
- added R150: 0, Resistor_SMD:R_0402_1005Metric, symbol Device:R
- added R151, R152: 100k, Resistor_SMD:R_0402_1005Metric, symbol Device:R
- added U10: TCAN1044VDRBRQ1, lcsc:VSON-8_L3.0-W3.0-P0.65-BR-EP, symbol lcsc_lib:TCAN1044VDRBRQ1
- added U24: SN74LVC2G66DCUR, lcsc:VSSOP-8_L2.1-W2.4-P0.50-LS3.2-BR, symbol lcsc_lib:SN74LVC2G66DCUR
- added U5: STM32H563ZIT6, lcsc:LQFP-144_L20.0-W20.0-P0.50-LS22.0-TL, symbol lcsc_lib:STM32H563ZIT6
- added U8: TPS2116DRLR, lcsc:SOT-583-8_L2.1-W1.6-P0.50-LS1.6-BL, symbol lcsc_lib:TPS2116DRLR
- added X1: SX3M48.000B10F20TNN, lcsc:OSC-SMD_4P-L3.2-W2.5-BL, symbol lcsc_lib:SX3M48.000B10F20TNN
- added Y2: Crystal_GND24, Crystal:Crystal_SMD_2016-4Pin_2.0x1.6mm, symbol Device:Crystal_GND24
- C1, C11, C13, C14, C25, C32, C36, C37, C38, C39, C4, C6, C7, C8, C9: footprint Capacitor_SMD:C_0603_1608Metric -> Capacitor_SMD:C_0402_1005Metric; LCSC C14663 -> C307331
- C10, C12, C17, C5: footprint Capacitor_SMD:C_0603_1608Metric -> Capacitor_SMD:C_0402_1005Metric; LCSC C15849 -> C1518208
- C18: value 15p -> 100n; LCSC C1548 -> C307331; MPN (none) -> CC0603KRX7R9BB104
- C19: value 15p -> 1u; LCSC C1548 -> C1518208; MPN (none) -> CL21B105KBFNNNE
- C20, C22, C23, C27: footprint Capacitor_SMD:C_0603_1608Metric -> Capacitor_SMD:C_0402_1005Metric; LCSC C14663 -> C307331; MPN (none) -> CC0603KRX7R9BB104
- C21: MFR GRM21BR61H106KE43L -> (none)
- C24, C26: value 100n -> 1u; footprint Capacitor_SMD:C_0603_1608Metric -> Capacitor_SMD:C_0402_1005Metric; LCSC C14663 -> C1518208; MPN (none) -> CL21B105KBFNNNE
- C33, C34: value 10u -> 100n; footprint Capacitor_SMD:C_0603_1608Metric -> Capacitor_SMD:C_0402_1005Metric; LCSC C96446 -> C307331; MFR GRM21BR61H106KE43L -> (none)
- C40, C41, C42: value 4.7u -> 100n; footprint Capacitor_SMD:C_0603_1608Metric -> Capacitor_SMD:C_0402_1005Metric; LCSC C19666 -> C307331
- R1: value 0 -> 47; footprint Resistor_SMD:R_0402_1005Metric -> Resistor_SMD:R_0603_1608Metric; JLC_DNF true -> (none); KiLib_Generator SMD_2terminal_chip_molded -> (none); LCSC C17168 -> C23182; now fitted; now in the parts list
- R13: value 0 -> 10k; LCSC C17168 -> C25744; now fitted; now in the parts list
- R18: JLC_DNF true -> (none); LCSC C17168 -> C25079; now fitted; now in the parts list
- TP3, TP7: now left out of the parts list
Connections:
- net A2D5 is gone; now on net LA_OUT2: U1.43 (IOT_49a)
- net A2D6 is gone; now on net LA_OUT1: U1.42 (IOT_51a)
- net A2D7 is gone; now on net LA_OUT4: U1.38 (IOT_50b)
- net A2D_CLK is gone; now on net LA_OUT3: U1.37 (IOT_45a_G1)
- net FLASH_SS_RP is gone; now on net ESP32_CS: R13.2
- net FPGA_ANALOG_OUTPUT is gone; now on net LA_OUT5: U1.36 (IOT_48b)
- net ICE_SWITCH_CONTROL is gone; now on net +3V3: R32.2
- net QSPI_CS_PSRAM is gone; now on net ICE_SS_PSRAM: R16.1
- net QSPI_SCLK is gone; now on net ICE_SCLK: U7.6 (SCLK)
- net QSPI_SD0 is gone; now on net ICE_SPI_SO: U7.5 (SI/SIO[0])
- net QSPI_SD1 is gone; now on net ICE_SPI_SI: U7.2 (SO/SIO[1])
- net QSPI_SD2 is gone; now on net ICE_IO2: U7.3 (SIO[2])
- net QSPI_SD3 is gone; now on net ICE_IO3: U7.7 (SIO[3])
- net XIN is gone; now on net GND: C18.1
- net +3V3: now also C20.2, C21.1, C22.2, C24.2, C26.2, C27.2, C33.1, C34.1, C40.1, C42.1, J1.17 (Pin_17), R13.1, R21.2, U7.8 (VDD), C121.1, C122.2, C220.1, C43.1, C52.2, C60.2, FB2.1, H1.1, LED1.2, R151.1, R152.1, R33.1, R35.2, U10.5 (NC/VIO), U24.8 (VCC), U5.106 (VDDUSB), U5.108 (VDD), U5.121 (VDDIO2), U5.131 (VDD), U5.144 (VDD), U5.17 (VDD), U5.30 (VDD), U5.39 (VDD), U5.52 (VDD), U5.6 (VBAT), U5.62 (VDD), U5.72 (VDD), U5.84 (VDD), U5.95 (VDD), U8.3 (VIN1), X1.1 (TRI-STATE), X1.4 (VDD); no longer C10.2, C14.2, C17.2, C20.1, C21.2, C22.1, C23.1, C24.1, C27.1, C33.2, C34.2, C8.2, J1.13 (Pin_13), J1.15 (Pin_15), U1.33 (VCCIO_0)
- net +5V: now also C14.2, C17.2, U10.3 (VCC)
- net CAN+: now also J1.19 (Pin_19), U10.7 (CANH), U24.1 (1A); no longer R18.1
- net CAN-: now also J1.20 (Pin_20), R18.1, U10.6 (CANL); no longer R18.2
- net ESP32_BOOT: now also U5.50 (PF12)
- net ESP32_EN: now also C10.2, U5.49 (PF11)
- net ESP32_RX: now also U5.101 (PA9)
- net ESP32_TX: now also U5.102 (PA10)
- net GND: now also C19.1, C20.1, C21.2, C22.1, C23.1, C24.1, C26.1, C27.1, C33.2, C34.2, J1.15 (Pin_15), R22.1, C121.2, C122.1, C218.2, C219.2, C220.2, C43.2, C48.1, C50.2, C51.2, C52.1, C53.1, C54.1, C55.1, C59.1, C60.1, H1.3, H1.5, H1.9, H2.6, R138.2, R34.1, R89.2, U10.2 (GND), U10.9 (EP), U24.4 (GND), U5.107 (VSS), U5.120 (VSS), U5.130 (VSS), U5.143 (VSS), U5.16 (VSS), U5.31 (VSSA), U5.38 (VSS), U5.51 (VSS), U5.61 (VSS), U5.71 (VSS), U5.83 (VSS), U5.94 (VSS), U8.1 (GND), U8.5 (MODE), X1.2 (GND), Y2.2 (G), Y2.4 (G); no longer C18.2, C19.2, C20.2, C21.1, C22.2, C23.2, C24.2, C26.2, C27.2, C33.1, C34.1, J1.14 (Pin_14), R21.2, R32.1
- net I2C0_SCL: now also U5.139 (PB8)
- net I2C0_SDA: now also U5.140 (PB9)
- net I2C1_SCL: now also H2.8, U5.11 (PF1)
- net I2C1_SDA: now also H2.7, U5.10 (PF0)
- net ICE_CDONE: now also U5.54 (PF14)
- net ICE_CRESET: now also U5.53 (PF13)
- net ICE_SCLK: now also U5.22 (PF10)
- net ICE_SPI_SI: now also U5.21 (PF9)
- net ICE_SPI_SO: now also U5.20 (PF8)
- net ICE_SS: now also U5.2 (PE3)
- net LA_OUT1: no longer U1.19 (IOB_29b)
- net LA_OUT10: now also U1.28 (IOT_41a); no longer U1.32 (IOT_43a)
- net LA_OUT11: now also U1.26 (IOT_39a); no longer U1.35 (IOT_46b_G0)
- net LA_OUT12: now also U1.27 (IOT_38b); no longer U1.34 (IOT_44b)
- net LA_OUT2: no longer U1.20 (IOB_25b_G3)
- net LA_OUT3: no longer U1.21 (IOB_23b)
- net LA_OUT4: no longer U1.23 (IOT_37a)
- net LA_OUT5: no longer U1.25 (IOT_36b)
- net LA_OUT6: now also U1.35 (IOT_46b_G0); no longer U1.26 (IOT_39a)
- net LA_OUT7: now also U1.34 (IOT_44b); no longer U1.27 (IOT_38b)
- net LA_OUT8: now also U1.32 (IOT_43a); no longer U1.28 (IOT_41a)
- net P_USB_D+: now also U5.104 (PA12)
- net P_USB_D-: now also U5.103 (PA11)
- net SWCLK: now also H1.4, U5.109 (PA14)
- net SWDIO: now also H1.2, U5.105 (PA13)
- net at C5.2, C6.2, FB1.2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: now also C48.2, C59.2
- net ICE_IO2: now reaches R4.2, U2.3 (/WP(IO2))
- net ICE_IO2: now also U1.20 (IOB_25b_G3), U5.19 (PF7)
- net ICE_IO3: now reaches R8.2, U2.7 (/HOLD_OR_/RESET(IO3))
- net ICE_IO3: now also U1.21 (IOB_23b), U5.18 (PF6)
- net at U1.41 (RGB2): now also LED1.4
- net ESP32_HANDSHAKE: now reaches U4.12 (IO0)
- net ESP32_HANDSHAKE: now also U5.46 (PB0)
- net ESP32_DATAREADY: now reaches U4.13 (IO1)
- net ESP32_DATAREADY: now also U5.47 (PB1)
- net ESP32_CS: now reaches U4.16 (IO10)
- net ESP32_CS: now also U5.48 (PB2)
- net ESP32_CTS: now reaches U4.19 (IO5)
- net ESP32_CTS: now also U5.63 (PE10)
- net ESP32_SCLK: now reaches U4.20 (IO6)
- net ESP32_SCLK: now also U5.65 (PE12)
- net ESP32_MOSI: now reaches U4.21 (IO7)
- net ESP32_MOSI: now also U5.67 (PE14)
- net ESP32_MISO: now reaches U4.5 (IO2)
- net ESP32_MISO: now also R33.2, U5.66 (PE13)
- net ESP32_RTS: now reaches U4.6 (IO3)
- net ESP32_RTS: now also U5.64 (PE11)
- net STM32_BOOT0: now reaches SW2.2
- net STM32_BOOT0: now also R34.2, U5.138 (BOOT0)
- net +1V8: now reaches J1.18 (Pin_18)
- net +1V8: now also U8.6 (VIN2)
- net at U1.39 (RGB0): now also LED1.1 (K)
- net at U1.40 (RGB1): now also LED1.3
- net at R12.1: now also U10.8 (STB)
- removed net +1V1: C26.1, C42.1
- net A2D0 renamed ICE_STM32_OTHER2
- net ICE_STM32_OTHER2: now also U5.55 (PF15)
- net A2D1 renamed ICE_STM32_OTHER1
- net ICE_STM32_OTHER1: now also U5.56 (PG0)
- net A2D2 renamed ICE_STM32_OTHER0
- net ICE_STM32_OTHER0: now also U5.57 (PG1)
- net A2D3 renamed ICE_SS_PSRAM
- net ICE_SS_PSRAM: now also U5.3 (PE4)
- net A2D4 renamed ICE_CLOCK
- net ICE_CLOCK: now also X1.3 (OUTPUT)
- net CAN_D renamed ADC_SDO
- net CAN_R renamed ADC_SCLK
- net FLASH_SS_ICE: no longer names the net of R2.2, R5.2, U2.1 (/CS)
- net FLASH_SS_ICE: no longer R1.2
- net GPIO0: no longer names the net of R1.1
- net GPIO0: now also C18.2, C19.2, FB2.2, U5.33 (VDDA); no longer R13.1
- net ICE_RP_CS0 renamed ICE_STM32_SCK
- net ICE_STM32_SCK: now also U5.41 (PA5)
- net ICE_RP_MISO renamed ADC_SDI
- net ICE_RP_MOSI renamed ICE_STM32_MISO
- net ICE_STM32_MISO: now also U5.42 (PA6)
- net ICE_RP_OTHER0 renamed ICE_STM32_MOSI
- net ICE_STM32_MOSI: now also U5.135 (PB5)
- net ICE_RP_OTHER1 renamed DAC_SYNC
- net ICE_RP_OTHER2 renamed DAC_SCLK
- net ICE_RP_OTHER3 renamed DAC_DIN
- net ICE_RP_SCK renamed ICE_STM32_CS0
- net ICE_STM32_CS0: now also R32.1, U5.69 (PB10)
- net QSPI_SS renamed NRST
- net NRST: now also C54.2, H1.10, R35.1, U5.25 (NRST)
- net SPI1_CS0 renamed SPI2_CS1
- net SPI2_CS1: now also H2.5, U5.59 (PE8)
- net SPI1_CS1 renamed SPI2_CS0
- net SPI2_CS0: now also H2.1, U5.60 (PE9)
- new net: C23.2, C55.2, R1.2, U5.32 (VREF+)
- new net: C219.1, U5.70 (VCAP)
- new net: R138.1, U24.3 (2C)
- new net: R18.2, U24.2 (1B)
- new net: C51.1, R150.2, Y2.3
- new net ADC_CNVST: U1.19 (IOB_29b)
- new net CAN_TERM_CTRL: R89.1, U24.7 (1C), U5.40 (PA4)
- new net EFUSE_INT: U5.100 (PA8)
- new net FDCAN1_RX: U10.4 (RXD), U5.114 (PD0)
- new net FDCAN1_TX: U10.1 (TXD), U5.115 (PD1)
- new net HEADER1_1: H3.1, U5.90 (PG5)
- new net HEADER1_10: H3.10, U5.77 (PD8)
- new net HEADER1_2: H3.2, U5.87 (PG2)
- new net HEADER1_3: H3.3, U5.86 (PD15)
- new net HEADER1_4: H3.4, U5.85 (PD14)
- new net HEADER1_5: H3.5, U5.82 (PD13)
- new net HEADER1_6: H3.6, U5.81 (PD12)
- new net HEADER1_7: H3.7, U5.80 (PD11)
- new net HEADER1_8: H3.8, U5.79 (PD10)
- new net HEADER1_9: H3.9, U5.78 (PD9)
- new net LA_INPUT13: J1.13 (Pin_13)
- new net LA_INPUT14: J1.14 (Pin_14)
- new net LA_OUT13: U1.25 (IOT_36b)
- new net LA_OUT14: U1.23 (IOT_37a)
- new net LA_VCCIO: C53.2, C8.2, U1.33 (VCCIO_0), U8.2 (VOUT), U8.7 (VOUT)
- new net LA_VCCIO_ST: R152.2, U5.89 (PG4), U8.8 (ST)
- new net LA_VCCIO_SWITCH: R151.2, U5.88 (PG3), U8.4 (PR1)
- new net PD7: U5.123 (PD7)
- new net PG10: U5.125 (PG10)
- new net PG9: U5.124 (PG9)
- new net PH0: C50.1, U5.23 (PH0-OSC_IN), Y2.1
- new net PH1: R150.1, U5.24 (PH1-OSC_OUT)
- new net RMII_CRS_DV: U5.43 (PA7)
- new net RMII_MDC: U5.27 (PC1)
- new net RMII_MDIO: U5.36 (PA2)
- new net RMII_NRST: U5.1 (PE2)
- new net RMII_REF_CLK: U5.35 (PA1)
- new net RMII_RXD0: U5.44 (PC4)
- new net RMII_RXD1: U5.45 (PC5)
- new net RMII_TXD0: U5.128 (PG13)
- new net RMII_TXD1: U5.76 (PB15)
- new net RMII_TX_EN: U5.126 (PG11)
- new net SPI2_MISO: H2.4, U5.75 (PB14)
- new net SPI2_MOSI: H2.3, U5.29 (PC3)
- new net SPI2_SCK: H2.2, U5.74 (PB13)
- new net STM32_VCAP1: C218.1, U5.142 (VCAP)
- new net USART2_RX: H2.10, U5.122 (PD6)
- new net USART2_TX: H2.9, U5.119 (PD5)
- no-connect marks 28 -> 58
Other:
- removed sheet analog to digital
- removed sheet digital to analog
- added sheet Analog Power v2 (analog-power-v2.kicad_sch)
- added sheet Ethernet (ethernet.kicad_sch)
- added sheet USB (usb.kicad_sch)
- added sheet analog switching (analog-switching.kicad_sch)
- added sheet analog to digital v2 (analog-to-digital-v2.kicad_sch)
- added sheet digital to analog v2 (digital-to-analog-v2.kicad_sch)
- sheet LogicAnalyzer ports: added A13, A14, OUT13, OUT14; removed none
- sheet Power ports: added EFUSE_INT, SCL, SDA; removed EFUSE1_ENABLE, EFUSE1_FLT, EFUSE1_V, EFUSE2_ENABLE, EFUSE2_FLT, EFUSE2_V, P_USB_D+, P_USB_D-
- note added: "25Mhz Crystal"
- note added: "Analog Power"
- note added: "Boot Button"
- note added: "Ethernet"
- note added: "QSPI: ICE flash and psram SPI1: ICE SPI SPI2: Header SPI SPI3: SPI4: esp32 SPI"
- note added: "Reset Button"
- note added: "STM32H563"
- note added: "USART1: esp32 USART2: header pins"
- note added: "USB"
- note removed: "12MHz Crystal"
- note removed: "Headers Switch for ICE SPI"
- note removed: "RP2350B"
- note removed: "RP2350B Flash"
- moved on the sheet: C10, C12, C14, C15, C16, C17, C25, C32, C36, C37, C38, C39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
