File: pcb/benchpod/vbench-pod.kicad_sch (KiCad schematic)
At the start: 116 parts, among them J1 PZ254V-12-22P, SW1 TS-1088-AR02016, SW2 TS-1088-AR02016, U1 ICE40UP5K-SG48ITR, U10 TCAN1044VDRBRQ1, U2 W25Q64JVSSIQ, U24 SN74LVC2G66DCUR, U28 SRV05-4.TCT, U4 ESP32-C3-MINI-1-N4, U5 STM32H563ZGT6, U7 APS6404L-3SQR-ZR, U8 TPS2116DRLR, X1 SX3M48.000B10F20TNN, Y2 6pF ±10ppm SMD2016-4P Crystal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

Commit message: header cleanup and schematic cleanup
Parts:
- removed H2: HC-PZ127-7.2L-2X5PZ, lcsc:HDR-TH_HC-PZ127-7.2L-2X5PZ, symbol lcsc_lib:HC-PZ127-7.2L-2X5PZ
- removed R27, R30: 10k, Resistor_SMD:R_0402_1005Metric, symbol Device:R
- removed R28, R29: 4.7k, Resistor_SMD:R_0402_1005Metric, symbol Device:R
Connections:
- net I2C1_SCL: no longer names the net of U5.11 (PF1)
- net I2C1_SDA: no longer names the net of U5.10 (PF0)
- net SPI2_CS0: no longer names the net of U5.60 (PE9)
- net SPI2_CS1: no longer names the net of U5.59 (PE8)
- net SPI2_MISO: no longer names the net of U5.75 (PB14)
- net SPI2_MOSI: no longer names the net of U5.29 (PC3)
- net SPI2_SCK: no longer names the net of U5.74 (PB13)
- net USART2_RX: no longer names the net of U5.122 (PD6)
- net USART2_TX: no longer names the net of U5.119 (PD5)
- no-connect marks 58 -> 67
