File: pcb/benchpod/vbench-pod.kicad_sch (KiCad schematic)
At the start: 113 parts, among them J1 PZ254V-12-22P, J10 TC2030-IDC, SW1 TS-1088-AR02016, SW2 TS-1088-AR02016, U1 ICE40UP5K-SG48ITR, U10 TCAN1044VDRBRQ1, U2 W25Q64JVSSIQ, U24 SN74LVC2G66DCUR, U28 SRV05-4.TCT, U4 ESP32-C3-MINI-1-N4, U5 STM32H563ZGT6, U7 APS6404L-3SQR-ZR, U8 TPS2116DRLR, X1 SX3M48.000B10F20TNN, Y2 6pF ±10ppm SMD2016-4P Crystal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

Commit message: pcb placement of v3r2 changes
Parts:
- removed J10: TC2030-IDC, Connector:Tag-Connect_TC2030-IDC-FP_2x03_P1.27mm_Vertical, symbol Connector:Conn_ARM_SWD_TagConnect_TC2030
- removed TP10: GND, TestPoint:TestPoint_Pad_1.5x1.5mm, symbol Connector:TestPoint
- removed TP8: USART2_TX, TestPoint:TestPoint_Pad_1.5x1.5mm, symbol Connector:TestPoint
- removed TP9: USART2_RX, TestPoint:TestPoint_Pad_1.5x1.5mm, symbol Connector:TestPoint
- added J10, J11: Conn_02x02_Counter_Clockwise, Connector_PinSocket_2.54mm:PinSocket_2x02_P2.54mm_Vertical, symbol Connector_Generic:Conn_02x02_Counter_Clockwise
Connections:
- net +3V3: now also J11.2 (Pin_2)
- net GND: now also J11.3 (Pin_3)
- net NRST: now also J10.2 (Pin_2)
- net SWCLK: now also J10.3 (Pin_3)
- net SWDIO: now also J10.4 (Pin_4)
- net SWO: now also J10.1 (Pin_1)
- net USART2_RX: now also J11.1 (Pin_1)
- net USART2_TX: now also J11.4 (Pin_4)

Commit message: esd fixes
Connections:
- net +1V8: no longer U28.4
- net LA_VCCIO: no longer U28.6
- no-connect marks 69 -> 71
Changed lines of the file:
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@@
 	)
 	(no_connect
+		(at 184.15 219.71)
+	)
+	(no_connect
 		(at 330.2 83.82)
 	)
@@
 	)
 	(no_connect
+		(at 184.15 214.63)
+	)
+	(no_connect
 		(at 173.99 105.41)
 	)
@@
 		)
 	)
-	(label "LA_VCCIO"
-		(at 184.15 219.71 180)
-		(effects
-			(font
-				(size 1.27 1.27)
-			)
-			(justify right bottom)
-		)
-	)
 	(label "ICE_SS_PSRAM"
 		(at 170.18 255.27 180)
@@
 		)
 	)
-	(label "+1V8"
-		(at 184.15 214.63 180)
-		(effects
-			(font
-				(size 1.27 1.27)
-			)
-			(justify right bottom)
-		)
-	)

Commit message: silkscreen fixes
Parts:
- J10, J11: now not fitted
Changed lines of the file:
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@@
 		(on_board yes)
 		(in_pos_files yes)
-		(dnp no)
+		(dnp yes)
 		(fields_autoplaced yes)
 		(property "Reference" "J11"
@@
 		(on_board yes)
 		(in_pos_files yes)
-		(dnp no)
+		(dnp yes)
 		(fields_autoplaced yes)
 		(property "Reference" "J10"
