File: pcb/benchpod/ethernet.kicad_sch (KiCad schematic)
At the start: 36 parts, among them J7 HR911105A_C12074, U6 LAN8742AI-CZ-TR, Y1 Crystal_GND24

Commit message: replacement for crystals, revision resistors, cleanups
Parts:
- Y1: LCSC C20623595 -> C49867546
Changed lines of the file:
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@@
 			)
 		)
-		(property "Description" "Four pin crystal, GND on pins 2 and 4"
+		(property "Description" "Four pin crystal, GND on pins 2 and 4. 25MHz/6pF, ESR ≤100Ω required (LAN8742A PHY ref clk on Y1"
 			(at 130.81 76.2 0)
 			(hide yes)
@@
 			)
 		)
-		(property "LCSC" "C20623595"
+		(property "LCSC" "C49867546"
 			(at 130.81 76.2 0)
 			(hide yes)

Commit message: replace d1, cleanups, cap changes
Parts:
- Y1: value Crystal_GND24 -> 6pF ±10ppm SMD2016-4P Crystals - 25Mhz
Changed lines of the file:
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@@
 			)
 		)
-		(property "Value" "Crystal_GND24"
+		(property "Value" "6pF ±10ppm SMD2016-4P Crystals  - 25Mhz"
 			(at 138.43 70.612 90)
 			(show_name no)

Commit message: fb changes, cc sensing, cleanups
Parts:
- FB3: footprint lcsc:L0603 -> lcsc_footprints:C85833_L0603; LCSC C1002 -> C85833
Changed lines of the file:
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@@
 			)
 		)
-		(property "Footprint" "lcsc:L0603"
+		(property "Footprint" "lcsc_footprints:C85833_L0603"
 			(at 117.602 33.02 90)
 			(hide yes)
@@
 			)
 		)
-		(property "LCSC" "C1002"
+		(property "LCSC" "C85833"
 			(at 119.38 33.02 0)
 			(hide yes)
