File: pcb/benchpod/ethernet.kicad_sch (KiCad schematic)
At the start: 36 parts, among them J7 HR911105A_C12074, U6 LAN8742AI-CZ-TR, Y1 6pF ±10ppm SMD2016-4P Crystal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

Commit message: analog v3r2: no extra BOM lines from the 0.1 % swaps and cap shrinks
JLC standard assembly charges per unique BOM line, so only keep changes
that replace a whole line:
- Revert 4.7 uF C2 C3 C5 C220 and 22 uF C16 C108 C154 C157 to 0805 (the
  other 4.7 uF/22 uF stay 0805, so the shrink split a line), and 5.1 pF C207
  C208 to the 0603 C2297586 (C140 needs it; 29 in stock = 9 boards).
- Move the remaining 1k (R21 R22 R164 R175), 1.5k (R15) and 2.2k (R58 R62)
  to the same 0.1 % parts as the precision ones, so their old lines go.

BOM: 122 -> 124 unique lines (0.1 % 10k for R109 R110 R111 R123, tantalum
C142). Netlist connectivity unchanged.

Co-Authored-By: Claude Opus 5.5 <noreply@anthropic.com>
Parts:
- R15: LCSC C25867 -> C281775
Changed lines of the file:
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@@
 			)
 		)
-		(property "LCSC" "C25867"
+		(property "LCSC" "C281775"
 			(at 41.91 97.79 0)
 			(hide yes)
