File: pcb/benchpod/usb.kicad_sch (KiCad schematic)
At the start: 27 parts, among them U57 TPS259470ARPWR

Commit message: Benchpod v3.0.1 work (#1)
* bom replacements and footprint replacements for out of stock items

* replacements and fixes

* smaller fixes

* finalized v3r1

* finshunt work on digital (wip)
Parts:
- added C103: 22u, Capacitor_SMD:C_0805_2012Metric, symbol Device:C
- added C260: 100n, Capacitor_SMD:C_0402_1005Metric, symbol Device:C
- added R138: 30m, Resistor_SMD:R_2512_6332Metric, symbol Device:R
- added U35: INA226, lcsc:VSSOP-10_L3.0-W3.0-P0.50-LS4.9-BL, symbol lcsc_lib:INA238AIDGSR
Connections:
- net +3V3: now also C260.2, U35.2 (A0), U35.6 (VS)
- net +5V: now also C103.1, R138.2, U35.8 (VBUS), U35.9 (IN-); no longer C225.2, C57.2, C91.1, C92.1, C93.1, D3.1 (K), U57.6 (OUT)
- net GND: now also C103.2, C260.1, U35.1 (A1), U35.7 (GND)
- new net +5V_IN: C225.2, C57.2, C91.1, C92.1, C93.1, D3.1 (K), R138.1, U35.10 (IN+), U57.6 (OUT)
- new net INA_SCL: U35.5 (SCL)
- new net INA_SDA: U35.4 (SDA)
- no-connect marks 4 -> 5
Other:
- note added: "Address 0x41"
- note added: "Current sensing BenchPod"
