File: pcb/benchpod/usb.kicad_sch (KiCad schematic)
At the start: 31 parts, among them U35 INA226, U57 TPS259470ARPWR

Commit message: analog v3r2: lead-free diodes and SMA, 0.1 % gain resistors, tantalum ADC reference cap
RoHS/REACH (no exemption claimed in the LCSC test reports):
- SS34 D3 D9 D15 D16 -> FOSAN SS34 C3014011
- SMAJ20A D5 -> FOSAN SMAJ20A C5353170
- SMAJ36CA D6 D7 D8 D10 -> FOSAN SMAJ36CA C5353135
- SMA RF1-RF4 -> HCTL HC-SMA-KWE-14.5H-D002-01 C41410437 (same footprint,
  5.08 vs 5.10 mm pin square)
- 11.8k R127 R129 R132 R133 (RALEC, lead glass) -> YAGEO 0.1 % C852496

0.1 % 25 ppm thin film, to cut the pod-to-pod offset and gain spread:
- THS4551 gain R92 R93 (1k C852624), R94 R102 (1.5k C281775): the 1 %
  mismatch turned VOCM into an ADC offset of about +-66 mV between pods
- +-12 V difference amps R126 R128 R130 R131 (2k C852711)
- VMID divider R110 R111, 3.3 V/5 V gains R108 (C861300), R109 R123
  (10k C190095), R122 (2.2k C326602)

C142 (MCP33131 VREF) 10 uF 0603 ceramic -> 10 uF tantalum case A C7171,
pin 1 (+) on AREF_4V096. Footprint change: needs a PCB update.

Netlist connectivity unchanged (pin-to-net diff identical), ERC unchanged.

Co-Authored-By: Claude Opus 5.5 <noreply@anthropic.com>
Parts:
- D3: LCSC C8678 -> C3014011; LCSC Part C8678 -> C3014011; Manufacturer MDD(辰达半导体) -> FOSAN
Changed lines of the file:
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@@
 			)
 		)
-		(property "Manufacturer" "MDD(辰达半导体)"
+		(property "Manufacturer" "FOSAN"
 			(at 124.46 142.24 0)
 			(hide yes)
@@
 			)
 		)
-		(property "LCSC Part" "C8678"
+		(property "LCSC Part" "C3014011"
 			(at 119.38 142.24 0)
 			(hide yes)
@@
 			)
 		)
-		(property "LCSC" "C8678"
+		(property "LCSC" "C3014011"
 			(at 137.16 142.24 90)
 			(hide yes)

Commit message: analog v3r2: smaller capacitor packages (same rating and dielectric)
To 0402: 3.3 nF C99 C102 C119 C226 (C26404), 8.2 pF C0G C29 C30 C50 C51
(C1579), 5.1 pF high-Q C207 C208 (C237535; the old C2297586 had 29 in stock).
To 0603: 4.7 uF C2 C3 C5 C220 (C69335), 22 uF C16 C108 C154 C157 (C2762594),
220 nF C189 (C64705), 2.2 uF X7R VCAP C218 C219 (C415535, from 1206).

Kept: C150/C153 (4.7 uF on the ~5 V charge-pump rails, DC-bias derating),
C140 (sees up to 58 V at TVS clamp), all 10 uF and the 22 uF on >5 V rails.
Footprint changes: needs a PCB update. Netlist connectivity unchanged.

Co-Authored-By: Claude Opus 5.5 <noreply@anthropic.com>
Parts:
- C226: footprint Capacitor_SMD:C_0603_1608Metric -> Capacitor_SMD:C_0402_1005Metric; LCSC C1613 -> C26404
Changed lines of the file:
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@@
 			)
 		)
-		(property "Footprint" "Capacitor_SMD:C_0603_1608Metric"
+		(property "Footprint" "Capacitor_SMD:C_0402_1005Metric"
 			(at 127.9652 101.6 0)
 			(hide yes)
@@
 			)
 		)
-		(property "LCSC" "C1613"
+		(property "LCSC" "C26404"
 			(at 127 97.79 0)
 			(hide yes)

Commit message: analog v3r2: EMC pre-scan fixes in the schematic, no new BOM lines
From compliance emc/prescan-2026-10-18.md (schematic part; layout is separate):
- C267 100 nF (C307331) at U37 (THS4551) pin 5 VS-; C224/C157 sit at the
  LM7705 on the power sheet, not at the driver.
- USB-C CC1/CC2 clamped by the two unused channels of D11 (USBLC6-4, pins
  6 and 4), which already protects D+/D-.
- LA header +1V8 (J1.18) and LA_VCCIO (J1.21) on the two unused channels of
  U28 (SRV05-4, pins 4 and 6); +3V3 (J1.17) is U28's own VDD rail, so it is
  clamped by U28 already. Layout: U28 next to J1.
- RF2 (0-5 V SMA) gets D21 SMF13CA (C1851355, same as D19/D20): the jack had
  no clamp of its own and floats behind K1 during cal1.
- CAN needs nothing: TCAN1044V is rated +-8 kV contact / +-15 kV air
  (system level) on CANH/CANL, plus the 56 ohm series resistors.

Netlist diff = exactly these connections; no field moves; ERC errors
unchanged (26); BOM 123 lines.

Co-Authored-By: Claude Opus 5.5 <noreply@anthropic.com>
Connections:
- net USB_CC2: now reaches R179.1, R75.2, USBC1.B5 (CC2)
- net USB_CC2: now also D11.4
- net USB_CC1: now reaches D11.6
- net USB_CC1: now also R178.1, R76.1, USBC1.A5 (CC1)
- no-connect marks 5 -> 3
Changed lines of the file:
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@@
-	)
-	(no_connect
-		(at 162.56 59.69)
 	)
 	(no_connect
@@
 		(at 243.84 133.35)
 	)
-	(no_connect
-		(at 162.56 41.91)
-	)
 	(wire
 		(pts
@@
 		)
 	)
+	(label "USB_CC2"
+		(at 162.56 59.69 0)
+		(effects
+			(font
+				(size 1.27 1.27)
+			)
+			(justify left bottom)
+		)
+	)
 	(label "INA_IN_P0"
 		(at 266.7 128.27 0)
@@
 		)
 	)
+	(label "USB_CC1"
+		(at 76.2 44.45 180)
+		(effects
+			(font
+				(size 1.27 1.27)
+			)
+			(justify right bottom)
+		)
+	)
 	(label "USB_D-"
 		(at 128.27 59.69 90)
@@
 		)
 	)
+	(label "USB_CC2"
+		(at 76.2 59.69 180)
+		(effects
+			(font
+				(size 1.27 1.27)
+			)
+			(justify right bottom)
+		)
+	)
 	(label "USB_D+"
 		(at 76.2 49.53 180)
@@
 		)
 	)
+	(label "USB_CC1"
+		(at 162.56 41.91 0)
+		(effects
+			(font
+				(size 1.27 1.27)
+			)
+			(justify left bottom)
+		)
+	)
