File: pcb/benchpod/analog-switching.kicad_sch (KiCad schematic)
At the start: 11 parts, among them U53 TPL7407LAPWR, U58 TCA9554PWR

Commit message: analog v3r2: +-14 V (TPS65131) enabled from U58 P4, off by default
U49 ENP/ENN were pulled up to VIN, so +-14 V was always on. They now share
the new ANA14_EN net from the relay expander U58 P4 (TCA9554 0x23, spare
pin), with R114 (100k) as pull-down to GND; R117 removed. TPS65131 EN:
VIH 1.4 V, 0.1 uA, so the 3.3 V expander output and 100k pull-down work.

Why: the DAC8554 powers up at code 0, which put the +-12 V output (RF3) at
about -12 V until firmware parked channel C. With +-14 V off at power-up,
-14 V is 0 V and +14 V sits at ~VIN - Vf (no BSW load switch), so U51
cannot swing negative and RF3 stays near 0 V. Old firmware never enables
it, so on v3r2 the +-12 V output is simply off. It also stops the
TPS65131 switching noise whenever the +-12 V output is not in use.

Firmware: on v3r2, park DAC channel C at mid-scale, then set U58 P4 high.
Netlist diff = exactly the intended changes; ERC errors unchanged (25);
BOM 123 lines.

Co-Authored-By: Claude Opus 5.5 <noreply@anthropic.com>
Connections:
- net ANA14_EN: now reaches U58.9 (P4)
- no-connect marks 7 -> 6
Changed lines of the file:
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@@
-	)
-	(no_connect
-		(at 96.52 62.23)
 	)
 	(no_connect
@@
 	(wire
 		(pts
+			(xy 96.52 62.23) (xy 104.14 62.23)
+		)
+		(stroke
+			(width 0)
+			(type default)
+		)
+	)
+	(wire
+		(pts
 			(xy 114.3 44.45) (xy 109.22 44.45)
 		)
@@
 		)
 	)
+	(hierarchical_label "ANA14_EN"
+		(shape output)
+		(at 104.14 62.23 0)
+		(effects
+			(font
+				(size 1.27 1.27)
+			)
+			(justify left)
+		)
+	)
