File: pcb/benchpod-digital/ethernet.kicad_sch (KiCad schematic)
At the start: 36 parts, among them J7 HR911105A_C12074, U6 LAN8742AI-CZ-TR, Y1 6pF ±10ppm SMD2016-4P Crystal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

Commit message: digital and analog cleanup
Parts:
- FB3: LCSC Part C1002 -> (none)
Changed lines of the file:
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@@
-			)
-		)
-		(property "LCSC Part" "C1002"
-			(at 119.38 33.02 0)
-			(hide yes)
-			(show_name no)
-			(do_not_autoplace no)
-			(effects
-				(font
-					(size 1.27 1.27)
-				)
 			)
 		)
