File: pcb/benchpod-digital/ethernet.kicad_sch (KiCad schematic)
At the start: 36 parts, among them J7 HR911105A_C12074, U6 LAN8742AI-CZ-TR, Y1 6pF ±10ppm SMD2016-4P Crystal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

Commit message: digital v3r3: carry over the analog v3r2 schematic changes
Same refs and nets as analog v3r1 in these areas, so the v3r2 fixes map 1:1.

- RoHS: D3 SS34 C8678 -> C3014011, D5 SMAJ20A C41376408 -> C5353170.
- U4 ESP32-C3-MINI-1-H4 (C2934569): the N4 is out of stock at JLC; same
  module, footprint and chip, 105 C rated.
- Package shrinks (whole BOM lines, no new lines): 8.2p C29/C30/C50/C51 and
  3.3n C99/C102/C119/C226 0603 -> 0402, 2.2u C218/C219 1206 -> 0603.
- EMC: D11 spare channels on USB CC1/CC2, U34 spares on +1V8 and LA_VCCIO.
- Debug: H1 (SWD 2x5) and H3 (HEADER1) removed; J10 SWO/NRST/SWCLK/SWDIO and
  J11 USART2_RX/+3V3/GND/USART2_TX 2x2, both DNP; PB3 = SWO, PD5/PD6 = USART2.

Not carried over: the 0.1 % resistors (on analog they only share lines with
the ADC parts) and the R164 revision strap (stays 1k: firmware runs the
digital board as v3). The PCB still needs Update PCB from Schematic.

Co-Authored-By: Claude Opus 5.5 <noreply@anthropic.com>
Parts:
- C29, C30: footprint Capacitor_SMD:C_0603_1608Metric -> Capacitor_SMD:C_0402_1005Metric; LCSC C1685 -> C1579
Changed lines of the file:
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@@
 			)
 		)
-		(property "Footprint" "Capacitor_SMD:C_0603_1608Metric"
+		(property "Footprint" "Capacitor_SMD:C_0402_1005Metric"
 			(at 140.6652 91.44 0)
 			(hide yes)
@@
 			)
 		)
-		(property "LCSC" "C1685"
+		(property "LCSC" "C1579"
 			(at 139.7 87.63 0)
 			(hide yes)
@@
 			)
 		)
-		(property "Footprint" "Capacitor_SMD:C_0603_1608Metric"
+		(property "Footprint" "Capacitor_SMD:C_0402_1005Metric"
 			(at 147.0152 80.01 0)
 			(hide yes)
@@
 			)
 		)
-		(property "LCSC" "C1685"
+		(property "LCSC" "C1579"
 			(at 146.05 76.2 0)
 			(hide yes)

Commit message: digital v3r3: merge three single-use resistor lines into existing ones
- CAN series resistors R18/R176: 56 ohm -> 49.9 ohm (C325388).
- RJ45 LED resistors R140/R141: 270 ohm 0603 -> 330 ohm 0402 (C25104); the
  LEDs get slightly dimmer.
- VDDA/VREF+ filter R1: 47 ohm 0603 -> 49.9 ohm 0402 (C325388).

Three BOM lines fewer. The MDIO pull-up R15 stays 1.5k (LAN8742A reference
value). R140, R141 and R1 change footprint: re-place them after Update PCB.

Co-Authored-By: Claude Opus 5.5 <noreply@anthropic.com>
Parts:
- R140, R141: value 270 -> 330; footprint Resistor_SMD:R_0603_1608Metric -> Resistor_SMD:R_0402_1005Metric; LCSC C22966 -> C25104
Changed lines of the file:
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@@
 			)
 		)
-		(property "Value" "270"
+		(property "Value" "330"
 			(at 195.58 92.7099 0)
 			(show_name no)
@@
 			)
 		)
-		(property "Footprint" "Resistor_SMD:R_0603_1608Metric"
+		(property "Footprint" "Resistor_SMD:R_0402_1005Metric"
 			(at 191.262 91.44 90)
 			(hide yes)
@@
 			)
 		)
-		(property "LCSC" "C22966"
+		(property "LCSC" "C25104"
 			(at 193.04 91.44 0)
 			(hide yes)
@@
 			)
 		)
-		(property "Value" "270"
+		(property "Value" "330"
 			(at 217.17 92.7099 0)
 			(show_name no)
@@
 			)
 		)
-		(property "Footprint" "Resistor_SMD:R_0603_1608Metric"
+		(property "Footprint" "Resistor_SMD:R_0402_1005Metric"
 			(at 212.852 91.44 90)
 			(hide yes)
@@
 			)
 		)
-		(property "LCSC" "C22966"
+		(property "LCSC" "C25104"
 			(at 214.63 91.44 0)
 			(hide yes)
