File: pcb/benchpod-digital/ethernet.kicad_sch (KiCad schematic)
At the start: 36 parts, among them J7 HR911105A_C12074, U6 LAN8742AI-CZ-TR, Y1 6pF ±10ppm SMD2016-4P Crystal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

Commit message: signal improvements
Parts:
- added R27: 33, Resistor_SMD:R_0402_1005Metric, symbol Device:R
Connections:
- net RMII_REF_CLK: now also R27.1; no longer U6.14 (nINT/REFCLKO)
- new net: R27.2, U6.14 (nINT/REFCLKO)
Changed lines of the file:
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@@
 	(wire
 		(pts
-			(xy 29.21 77.47) (xy 43.18 77.47)
+			(xy 29.21 77.47) (xy 31.75 77.47)
 		)
 		(stroke
@@
 	(wire
 		(pts
+			(xy 39.37 77.47) (xy 43.18 77.47)
+		)
+		(stroke
+			(width 0)
+			(type default)
+		)
+	)
+	(wire
+		(pts
 			(xy 130.81 80.01) (xy 135.89 80.01)
 		)
@@
 	(wire
 		(pts
-			(xy 27.94 80.01) (xy 43.18 80.01)
+			(xy 27.94 88.9) (xy 34.29 88.9)
 		)
 		(stroke
@@
 	(wire
 		(pts
+			(xy 34.29 88.9) (xy 43.18 80.01)
+		)
+		(stroke
+			(width 0)
+			(type default)
+		)
+	)
+	(wire
+		(pts
 			(xy 193.04 76.2) (xy 193.04 87.63)
 		)
@@
 	(hierarchical_label "RMII_MDC"
 		(shape input)
-		(at 27.94 80.01 180)
+		(at 27.94 88.9 180)
 		(effects
 			(font
@@
 					(unit 1)
 				)
+			)
+		)
+	)
+	(symbol
+		(lib_id "Device:R")
+		(at 35.56 77.47 90)
+		(unit 1)
+		(body_style 1)
+		(exclude_from_sim no)
+		(in_bom yes)
+		(on_board yes)
+		(in_pos_files yes)
+		(dnp no)
+		(property "Reference" "R27"
+			(at 35.56 79.756 90)
+			(show_name no)
+			(do_not_autoplace no)
+			(effects
+				(font
+					(size 1.27 1.27)
+				)
+			)
+		)
+		(property "Value" "33"
+			(at 35.56 82.296 90)
+			(show_name no)
+			(do_not_autoplace no)
+			(effects
+				(font
+					(size 1.27 1.27)
+				)
+			)
+		)
+		(property "Footprint" "Resistor_SMD:R_0402_1005Metric"
+			(at 35.56 79.248 90)
+			(hide yes)
+			(show_name no)
+			(do_not_autoplace no)
+			(effects
+				(font
+					(size 1.27 1.27)
+				)
+			)
+		)
+		(property "Datasheet" ""
+			(at 35.56 77.47 0)
+			(hide yes)
+			(show_name no)
+			(do_not_autoplace no)
+			(effects
+				(font
+					(size 1.27 1.27)
+				)
+			)
+		)
+		(property "Description" "Resistor"
+			(at 35.56 77.47 0)
+			(hide yes)
+			(show_name no)
+			(do_not_autoplace no)
+			(effects
+				(font
+					(size 1.27 1.27)
+				)
+			)
+		)
+		(property "LCSC" "C25105"
+			(at 35.56 77.47 90)
+			(hide yes)
+			(show_name no)
+			(do_not_autoplace no)
+			(effects
+				(font
+					(size 1.27 1.27)
+				)
+			)
+		)
+		(property "ProductID" ""
+			(at 35.56 77.47 90)
+			(hide yes)
+			(show_name no)
+			(do_not_autoplace no)
+			(effects
+				(font
+					(size 1.27 1.27)
+				)
+			)
+		)
+		(property "Sim.Pins" ""
+			(at 35.56 77.47 90)
+			(hide yes)
+			(show_name no)
+			(do_not_autoplace no)
+			(effects
+				(font
+					(size 1.27 1.27)
+				)
+			)
+		)
+		(property "KLC_S3.3" ""
+			(at 35.56 77.47 90)
+			(hide yes)
+			(show_name no)
+			(do_not_autoplace no)
+			(effects
+				(font
+					(size 1.27 1.27)
+				)
+			)
+		)
+		(property "KLC_S4.1" ""
+			(at 35.56 77.47 90)
+			(hide yes)
+			(show_name no)
+			(do_not_autoplace no)
+			(effects
+				(font
+					(size 1.27 1.27)
+				)
+			)
+		)
+		(pin "1"
+		)
+		(pin "2"
+		)
+		(instances
+			(project "vbench-pod"
+				(path "/745fcf4b-2e0b-4fc4-95c0-f2e3fd40beb9/0c40e001-2f3c-4e38-99cd-bf6c5858d9e0"
+					(reference "R27")
+					(unit 1)
+				)

Commit message: signal improvements
Changed lines of the file:
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@@
 	)
 	(junction
-		(at 184.15 72.39)
-		(diameter 0)
-		(color 0 0 0 0)
-	)
-	(junction
 		(at 81.28 20.32)
 		(diameter 0)
@@
 	(wire
 		(pts
-			(xy 184.15 72.39) (xy 214.63 72.39)
+			(xy 184.15 80.01) (xy 185.42 80.01)
 		)
 		(stroke
@@
 	(wire
 		(pts
-			(xy 181.61 72.39) (xy 184.15 72.39)
-		)
-		(stroke
-			(width 0)
-			(type default)
-		)
-	)
-	(wire
-		(pts
 			(xy 130.81 72.39) (xy 146.05 72.39)
 		)
@@
 	(wire
 		(pts
+			(xy 185.42 80.01) (xy 185.42 72.39)
+		)
+		(stroke
+			(width 0)
+			(type default)
+		)
+	)
+	(wire
+		(pts
 			(xy 214.63 87.63) (xy 214.63 82.55)
 		)
@@
 	(wire
 		(pts
-			(xy 184.15 87.63) (xy 184.15 72.39)
+			(xy 184.15 87.63) (xy 184.15 80.01)
 		)
 		(stroke
@@
 	(wire
 		(pts
+			(xy 185.42 72.39) (xy 214.63 72.39)
+		)
+		(stroke
+			(width 0)
+			(type default)
+		)
+	)
+	(wire
+		(pts
 			(xy 113.03 80.01) (xy 113.03 82.55)
 		)
@@
 	)
 	(label "GREEN_LED"
-		(at 181.61 72.39 180)
+		(at 184.15 80.01 180)
 		(effects
 			(font
@@
 		)
 		(property "Value" "6pF ±10ppm SMD2016-4P Crystals  - 25Mhz"
-			(at 138.43 70.612 90)
+			(at 170.434 70.104 90)
 			(show_name no)
 			(do_not_autoplace no)
