File: pcb/benchpod-digital/ethernet.kicad_sch (KiCad schematic)
At the start: 40 parts, among them J7 HR911105A_C12074, U6 LAN8742AI-CZ-TR, Y1 6pF ±10ppm SMD2016-4P Crystal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

Commit message: signal filtering / improvement
Connections:
- net RXN: now also D4.4 (D2+), D4.7 (NC); no longer D4.5 (D2-), D4.6 (NC)
- net RXP: now also D4.5 (D2-), D4.6 (NC); no longer D4.4 (D2+), D4.7 (NC)
- net TXN: now also D4.1 (D1+), D4.10 (NC); no longer D4.2 (D1-), D4.9 (NC)
- net TXP: now also D4.2 (D1-), D4.9 (NC); no longer D4.1 (D1+), D4.10 (NC)
