File: pcb/benchpod-digital/power.kicad_sch (KiCad schematic)
At the start: 70 parts, among them J4 Screw_Terminal_01x02, J5 Screw_Terminal_01x02, J6 Screw_Terminal_01x02, U26 TPS259470ARPWR, U27 TPS259470ARPWR, U29 INA238AIDGSR, U30 TPS82130SILR, U31 AP2112K-1.2, U32 AP2112K-2.5TRG1, U33 INA238AIDGSR, U52 AP2112K-1.8TRG1, U56 TCA9554PWR

Commit message: digital and analog cleanup
Parts:
- R83: value 50m -> 30m; LCSC C5200068 -> C2941066
- R84: value 30m -> 20m; LCSC C2941066 -> C915979
- U29, U33: value INA238AIDGSR -> INA226AIDGSR; LCSC C2868250 -> C49851; LCSC Part C2868250 -> C49851; MPN INA238AIDGSR -> (none); Manufacturer TI(德州仪器) -> (none)
Changed lines of the file:
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@@
 			)
 		)
-		(property "Value" "INA238AIDGSR"
+		(property "Value" "INA226AIDGSR"
 			(at 259.08 140.97 0)
 			(show_name no)
@@
 			)
 		)
-		(property "Datasheet" "https://www.lcsc.com/datasheet/C2868250.pdf"
+		(property "Datasheet" "https://www.lcsc.com/datasheet/C49851.pdf"
 			(at 259.08 166.37 0)
 			(hide yes)
@@
 			)
 		)
-		(property "Manufacturer" "TI(德州仪器)"
-			(at 259.08 168.91 0)
-			(hide yes)
-			(show_name no)
-			(do_not_autoplace no)
-			(effects
-				(font
-					(size 1.27 1.27)
-				)
-			)
-		)
-		(property "MPN" "INA238AIDGSR"
-			(at 259.08 171.45 0)
-			(hide yes)
-			(show_name no)
-			(do_not_autoplace no)
-			(effects
-				(font
-					(size 1.27 1.27)
-				)
-			)
-		)
-		(property "LCSC Part" "C2868250"
+		(property "LCSC Part" "C49851"
 			(at 259.08 173.99 0)
 			(hide yes)
@@
 			)
 		)
-		(property "LCSC" "C2868250"
+		(property "LCSC" "C49851"
 			(at 259.08 151.13 0)
 			(hide yes)
@@
 			)
 		)
-		(property "Value" "30m"
+		(property "Value" "20m"
 			(at 163.83 127 90)
 			(show_name no)
@@
 			)
 		)
-		(property "LCSC" "C2941066"
+		(property "LCSC" "C915979"
 			(at 163.83 129.54 90)
 			(hide yes)
@@
 			)
 		)
-		(property "Value" "50m"
+		(property "Value" "30m"
 			(at 161.29 90.17 90)
 			(show_name no)
@@
 			)
 		)
-		(property "LCSC" "C5200068"
+		(property "LCSC" "C2941066"
 			(at 161.29 92.71 90)
 			(hide yes)
@@
 			)
 		)
-		(property "Value" "INA238AIDGSR"
+		(property "Value" "INA226AIDGSR"
 			(at 207.01 142.24 0)
 			(show_name no)
@@
 			)
 		)
-		(property "Manufacturer" "TI(德州仪器)"
-			(at 207.01 170.18 0)
-			(hide yes)
-			(show_name no)
-			(do_not_autoplace no)
-			(effects
-				(font
-					(size 1.27 1.27)
-				)
-			)
-		)
-		(property "MPN" "INA238AIDGSR"
-			(at 207.01 172.72 0)
-			(hide yes)
-			(show_name no)
-			(do_not_autoplace no)
-			(effects
-				(font
-					(size 1.27 1.27)
-				)
-			)
-		)
-		(property "LCSC Part" "C2868250"
+		(property "LCSC Part" "C49851"
 			(at 207.01 175.26 0)
 			(hide yes)
@@
 			)
 		)
-		(property "LCSC" "C2868250"
+		(property "LCSC" "C49851"
 			(at 207.01 152.4 0)
 			(hide yes)

Commit message: finshunt work on digital (wip)
Connections:
- net +5V: no longer C94.2, C95.1, R67.1, U26.5 (IN)
- new net +5V_IN: C94.2, C95.1, R67.1, U26.5 (IN)
Changed lines of the file:
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@@
 			)
 		)
-		(property "Value" "+5V"
+		(property "Value" "+5V_IN"
 			(at 13.97 96.012 0)
 			(show_name no)
