File: pcb/benchpod-digital/power.kicad_sch (KiCad schematic)
At the start: 73 parts, among them J4 DB2ERC-3.81-2P-BK, J5 DB2ERC-3.81-2P-BK, J6 DB2ERC-3.81-2P-BK, U26 TPS259470ARPWR, U27 TPS259470ARPWR, U29 INA226AIDGSR, U30 TPS62130ARGTR, U31 AP2112K-1.2, U32 AP2112K-2.5TRG1, U33 INA226AIDGSR, U52 AP2112K-1.8TRG1, U56 TCA9554PWR

Commit message: pcb work
Parts:
- U30: footprint Package_DFN_QFN:VQFN-16-1EP_3x3mm_P0.5mm_EP1.68x1.68mm_ThermalVias -> lcsc_footprints:C337502_VQFN-16_L3_0-W3_0-P0_50-BL-EP1_7
