File: pcb/benchpod-digital/power.kicad_sch (KiCad schematic)
At the start: 73 parts, among them J4 DB2ERC-3.81-2P-BK, J5 DB2ERC-3.81-2P-BK, J6 DB2ERC-3.81-2P-BK, U26 TPS259470ARPWR, U27 TPS259470ARPWR, U29 INA226AIDGSR, U30 TPS62130ARGTR, U31 AP2112K-1.2, U32 AP2112K-2.5TRG1, U33 INA226AIDGSR, U52 AP2112K-1.8TRG1, U56 TCA9554PWR

Commit message: digital v3r3: EMC changes from vendor references
Ethernet (Microchip LAN8742A datasheet Fig. 3-23 + EVB8742, HanRun
HR911105A note, TI DP83825 EVM):
- R160 1M -> 0R 0402: J7 pin 8 (CHS GND) straight to GND; C58 DNP
- J7 center taps on their own net ETH_CT, fed from VDDA by R196 0R;
  C49 100n now sits on ETH_CT (place it at J7 pins 4/5)
- C273-C276 8.2p from TXP/TXN/RXP/RXN to GND (EVB8742 10 pF EMI option)

Power terminals (TI TPS25947EVM):
- 100n + 470p at J5 (C277/C278), J6 (C279/C280), J4 (C281/C282)
- J4 pin 1 net named EXT_IN

No new BOM lines. ERC unchanged (467 before and after).

Co-Authored-By: Claude Opus 5.5 <noreply@anthropic.com>
Parts:
- added C277, C279, C281: 100n, Capacitor_SMD:C_0402_1005Metric, symbol Device:C
- added C278, C280, C282: 470p, Capacitor_SMD:C_0402_1005Metric, symbol Device:C
Connections:
- net GND: now also C277.2, C278.2, C279.2, C280.2, C281.2, C282.2
- net INA_IN_M1: now also C277.1, C278.1
- net INA_IN_M2: now also C279.1, C280.1
- net EXT_IN: now reaches C62.1, C63.1, C96.2, D5.1, J4.1 (Pin_1), R70.1, U27.5 (IN)
- net EXT_IN: now also C281.1, C282.1
