File: pcb/benchpod-digital/usb.kicad_sch (KiCad schematic)
At the start: 28 parts, among them U57 TPS259470ARPWR

Commit message: digital and analog cleanup
Parts:
- removed D2: SS34, lcsc:SMA_L4.3-W2.6-LS5.2-RD, symbol lcsc_lib:SS34_C8678
Changed lines of the file:
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@@
 	)
 	(junction
-		(at 74.93 148.59)
-		(diameter 0)
-		(color 0 0 0 0)
-	)
-	(junction
 		(at 153.67 115.57)
 		(diameter 0)
@@
 		(color 0 0 0 0)
 	)
-	(junction
-		(at 118.11 137.16)
-		(diameter 0)
-		(color 0 0 0 0)
-	)
 	(no_connect
 		(at 162.56 59.69)
@@
 	(wire
 		(pts
-			(xy 74.93 148.59) (xy 118.11 148.59)
-		)
-		(stroke
-			(width 0)
-			(type default)
-		)
-	)
-	(wire
-		(pts
 			(xy 36.83 59.69) (xy 76.2 59.69)
 		)
@@
 	(wire
 		(pts
-			(xy 118.11 148.59) (xy 118.11 147.32)
-		)
-		(stroke
-			(width 0)
-			(type default)
-		)
-	)
-	(wire
-		(pts
 			(xy 68.58 62.23) (xy 76.2 62.23)
 		)
@@
 	(wire
 		(pts
-			(xy 118.11 137.16) (xy 137.16 137.16)
+			(xy 116.84 137.16) (xy 137.16 137.16)
 		)
 		(stroke
@@
 	(wire
 		(pts
-			(xy 116.84 137.16) (xy 118.11 137.16)
-		)
-		(stroke
-			(width 0)
-			(type default)
-		)
-	)
-	(wire
-		(pts
 			(xy 29.21 86.36) (xy 43.18 86.36)
 		)
@@
 					(unit 1)
 				)
-			)
-		)
-	)
-	(symbol
-		(lib_id "lcsc_lib:SS34_C8678")
-		(at 118.11 142.24 270)
-		(mirror x)
-		(unit 1)
-		(body_style 1)
-		(exclude_from_sim no)
-		(in_bom yes)
-		(on_board yes)
-		(in_pos_files yes)
-		(dnp no)
-		(property "Reference" "D2"
-			(at 113.538 141.224 90)
-			(show_name no)
-			(do_not_autoplace no)
-			(effects
-				(font
-					(size 1.27 1.27)
-				)
-				(justify right)
-			)
-		)
-		(property "Value" "SS34"
-			(at 113.538 143.764 90)
-			(show_name no)
-			(do_not_autoplace no)
-			(effects
-				(font
-					(size 1.27 1.27)
-				)
-				(justify right)
-			)
-		)
-		(property "Footprint" "lcsc:SMA_L4.3-W2.6-LS5.2-RD"
-			(at 110.49 142.24 0)
-			(hide yes)
-			(show_name no)
-			(do_not_autoplace no)
-			(effects
-				(font
-					(size 1.27 1.27)
-				)
-			)
-		)
-		(property "Datasheet" "https://lcsc.com/product-detail/Schottky-Barrier-Diodes-SBD_SS34_C8678.html"
-			(at 107.95 142.24 0)
-			(hide yes)
-			(show_name no)
-			(do_not_autoplace no)
-			(effects
-				(font
-					(size 1.27 1.27)
-				)
-			)
-		)
-		(property "Description" "SS34"
-			(at 118.11 142.24 0)
-			(hide yes)
-			(show_name no)
-			(do_not_autoplace no)
-			(effects
-				(font
-					(size 1.27 1.27)
-				)
-			)
-		)
-		(property "Manufacturer" "MDD(辰达半导体)"
-			(at 105.41 142.24 0)
-			(hide yes)
-			(show_name no)
-			(do_not_autoplace no)
-			(effects
-				(font
-					(size 1.27 1.27)
-				)
-			)
-		)
-		(property "MPN" "SS34"
-			(at 102.87 142.24 0)
-			(hide yes)
-			(show_name no)
-			(do_not_autoplace no)
-			(effects
-				(font
-					(size 1.27 1.27)
-				)
-			)
-		)
-		(property "LCSC Part" "C8678"
-			(at 100.33 142.24 0)
-			(hide yes)
-			(show_name no)
-			(do_not_autoplace no)
-			(effects
-				(font
-					(size 1.27 1.27)
-				)
-			)
-		)
-		(property "ProductID" ""
-			(at 118.11 142.24 90)
-			(hide yes)
-			(show_name no)
-			(do_not_autoplace no)
-			(effects
-				(font
-					(size 1.27 1.27)
-				)
-			)
-		)
-		(property "Sim.Pins" ""
-			(at 118.11 142.24 90)
-			(hide yes)
-			(show_name no)
-			(do_not_autoplace no)
-			(effects
-				(font
-					(size 1.27 1.27)
-				)
-			)
-		)
-		(property "KLC_S3.3" ""
-			(at 118.11 142.24 90)
-			(hide yes)
-			(show_name no)
-			(do_not_autoplace no)
-			(effects
-				(font
-					(size 1.27 1.27)
-				)
-			)
-		)
-		(property "KLC_S4.1" ""
-			(at 118.11 142.24 90)
-			(hide yes)
-			(show_name no)
-			(do_not_autoplace no)
-			(effects
-				(font
-					(size 1.27 1.27)
-				)
-			)
-		)
-		(property "LCSC" "C8678"
-			(at 118.11 142.24 90)
-			(hide yes)
-			(show_name no)
-			(do_not_autoplace no)
-			(effects
-				(font
-					(size 1.27 1.27)
-				)
-			)
-		)
-		(pin "1"
-		)
-		(pin "2"
-		)
-		(instances
-			(project "vbench-pod"
-				(path "/745fcf4b-2e0b-4fc4-95c0-f2e3fd40beb9/6e16e19c-a558-4ab3-b333-eb07c45a4c12"
-					(reference "D2")
-					(unit 1)
-				)

Commit message: finshunt work on digital (wip)
Parts:
- added C103: 22u, Capacitor_SMD:C_0805_2012Metric, symbol Device:C
- added C260: 100n, Capacitor_SMD:C_0402_1005Metric, symbol Device:C
- added R138: 30m, Resistor_SMD:R_2512_6332Metric, symbol Device:R
- added U35: INA226, lcsc:VSSOP-10_L3.0-W3.0-P0.50-LS4.9-BL, symbol lcsc_lib:INA238AIDGSR
Connections:
- net +3V3: now also C260.2, U35.2 (A0), U35.6 (VS)
- net +5V: now also C103.1, R138.2, U35.8 (VBUS), U35.9 (IN-); no longer C225.2, C57.2, C91.1, C92.1, C93.1, D3.1 (K), U57.6 (OUT)
- net GND: now also C103.2, C260.1, U35.1 (A1), U35.7 (GND)
- new net +5V_IN: C225.2, C57.2, C91.1, C92.1, C93.1, D3.1 (K), R138.1, U35.10 (IN+), U57.6 (OUT)
- new net INA_SCL: U35.5 (SCL)
- new net INA_SDA: U35.4 (SDA)
- no-connect marks 4 -> 5
Other:
- note added: "Address 0x41"
- note added: "Current sensing BenchPod"
