File: pcb/benchpod-digital/usb.kicad_sch (KiCad schematic)
At the start: 31 parts, among them U35 INA226AIDGSR, U57 TPS259470ARPWR

Commit message: bom changes, cleanups
Parts:
- D1: value SMAJ5.0A_C2925443 -> SMAJ5.0A
Changed lines of the file:
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@@
 			)
 		)
-		(property "Value" "SMAJ5.0A_C2925443"
+		(property "Value" "SMAJ5.0A"
 			(at 48.26 82.55 0)
 			(show_name no)
