File: pcb/benchpod-digital/module-link.kicad_sch (KiCad schematic)
At the start: 31 parts, among them CN1 KH-FPC1.0-H2.0SMT-24P-QCHF, U59 TPS259470ARPWR, U60 TPS259470ARPWR

Commit message: more pcb work
Connections:
- net MOD_ADC_SCLK: now also CN1.12; no longer CN1.11
- net MOD_ADC_SDI: now also CN1.11; no longer CN1.13
- net MOD_ADC_SDO: now also CN1.13; no longer CN1.12
- net MOD_DAC_DIN: now also CN1.7; no longer CN1.8
- net MOD_DAC_SCLK: now also CN1.8; no longer CN1.7
Changed lines of the file:
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@@
+		)
+	)
+	(hierarchical_label "MOD_DAC_SCLK"
+		(shape output)
+		(at 195.58 92.71 180)
+		(effects
+			(font
+				(size 1.27 1.27)
+			)
+			(justify right)
 		)
 	)
@@
 		)
 	)
+	(hierarchical_label "MOD_ADC_SCLK"
+		(shape output)
+		(at 195.58 102.87 180)
+		(effects
+			(font
+				(size 1.27 1.27)
+			)
+			(justify right)
+		)
+	)
 	(hierarchical_label "MOD_PWR_PG"
 		(shape input)
@@
 		)
 	)
+	(hierarchical_label "MOD_DAC_DIN"
+		(shape output)
+		(at 195.58 90.17 180)
+		(effects
+			(font
+				(size 1.27 1.27)
+			)
+			(justify right)
+		)
+	)
+	(hierarchical_label "BRIDGE_PWR_PG"
+		(shape input)
+		(at 154.94 59.69 270)
+		(effects
+			(font
+				(size 1.27 1.27)
+			)
+			(justify right)
+		)
+	)
+	(hierarchical_label "MOD_I2C_SDA"
+		(shape bidirectional)
+		(at 170.18 44.45 270)
+		(effects
+			(font
+				(size 1.27 1.27)
+			)
+			(justify right)
+		)
+	)
 	(hierarchical_label "MOD_ADC_SDO"
 		(shape input)
-		(at 195.58 102.87 180)
-		(effects
-			(font
-				(size 1.27 1.27)
-			)
-			(justify right)
-		)
-	)
-	(hierarchical_label "MOD_DAC_DIN"
-		(shape output)
-		(at 195.58 92.71 180)
+		(at 195.58 105.41 180)
+		(effects
+			(font
+				(size 1.27 1.27)
+			)
+			(justify right)
+		)
+	)
+	(hierarchical_label "MOD_RESET#"
+		(shape output)
+		(at 195.58 123.19 180)
+		(effects
+			(font
+				(size 1.27 1.27)
+			)
+			(justify right)
+		)
+	)
+	(hierarchical_label "MOD_PWR_EN"
+		(shape output)
+		(at 63.5 59.69 270)
+		(effects
+			(font
+				(size 1.27 1.27)
+			)
+			(justify right)
+		)
+	)
+	(hierarchical_label "MOD_I2C_SCL"
+		(shape bidirectional)
+		(at 185.42 44.45 270)
 		(effects
 			(font
@@
 	(hierarchical_label "MOD_ADC_SDI"
 		(shape output)
-		(at 195.58 105.41 180)
-		(effects
-			(font
-				(size 1.27 1.27)
-			)
-			(justify right)
-		)
-	)
-	(hierarchical_label "BRIDGE_PWR_PG"
-		(shape input)
-		(at 154.94 59.69 270)
-		(effects
-			(font
-				(size 1.27 1.27)
-			)
-			(justify right)
-		)
-	)
-	(hierarchical_label "MOD_DAC_SCLK"
-		(shape output)
-		(at 195.58 90.17 180)
-		(effects
-			(font
-				(size 1.27 1.27)
-			)
-			(justify right)
-		)
-	)
-	(hierarchical_label "MOD_ADC_SCLK"
-		(shape output)
 		(at 195.58 100.33 180)
 		(effects
 			(font
-				(size 1.27 1.27)
-			)
-			(justify right)
-		)
-	)
-	(hierarchical_label "MOD_I2C_SDA"
-		(shape bidirectional)
-		(at 170.18 44.45 270)
-		(effects
-			(font
-				(size 1.27 1.27)
-			)
-			(justify right)
-		)
-	)
-	(hierarchical_label "MOD_RESET#"
-		(shape output)
-		(at 195.58 123.19 180)
-		(effects
-			(font
-				(size 1.27 1.27)
-			)
-			(justify right)
-		)
-	)
-	(hierarchical_label "MOD_PWR_EN"
-		(shape output)
-		(at 63.5 59.69 270)
-		(effects
-			(font
-				(size 1.27 1.27)
-			)
-			(justify right)
-		)
-	)
-	(hierarchical_label "MOD_I2C_SCL"
-		(shape bidirectional)
-		(at 185.42 44.45 270)
-		(effects
-			(font
