File: pcb/benchpod-digital/module-link.kicad_sch (KiCad schematic)
At the start: 31 parts, among them CN1 KH-FPC1.0-H2.0SMT-24P-QCHF, U59 TPS259470ARPWR, U60 TPS259470ARPWR

Commit message: digital v3r3: SY6280AAC power switches for module and bridge, TVS on 5 V outputs
- U59 (module 5 V) and U60 (bridge USB-A 5 V) become SY6280AAC (C55136,
  about $0.09) instead of TPS259470 eFuses (about $1 each); 12 support parts
  removed. Current limit 6800/Rset: module 4.7k = about 1.45 A, bridge
  4.7k + 2.2k (R187 + R195) = 6.9k = about 1 A, both from existing BOM lines.
  EN keeps its 10k pull-up (on at power-up), PD10 / PD14 still switch them.
- The FLT/PG flags are gone with the eFuses: PD11, PD12, PD15 and PG2 are free
  again (no-connect), and their four sheet pins are removed.
- SMAJ5.0A TVS (same line as D1): D22 on the bridge USB-A VBUS, D23 on target
  power 1 (USB1/J5).

BOM: one new line (SY6280AAC). The TPS259470 line stays for U26, U27, U57.

Co-Authored-By: Claude Opus 5.5 <noreply@anthropic.com>
Parts:
- removed C261, C267: 10n, Capacitor_SMD:C_0402_1005Metric, symbol Device:C
- removed C262, C268: 3.3n, Capacitor_SMD:C_0402_1005Metric, symbol Device:C
- removed R181, R188: 37.4k, Resistor_SMD:R_0402_1005Metric, symbol Device:R
- removed R182, R184, R185, R189, R191, R192: 10k, Resistor_SMD:R_0402_1005Metric, symbol Device:R
- removed U59, U60: TPS259470ARPWR, lcsc:VQFN-10_L2.0-W2.0-P0.45-TL, symbol lcsc_lib:TPS259470ARPWR
- added D22: SMAJ5.0A_C2925443, lcsc:SMA_L4.3-W2.6-LS5.0-RD, symbol lcsc_lib:SMAJ5.0A_C2925443
- added R195: 2.2k, Resistor_SMD:R_0402_1005Metric, symbol Device:R
- added U59, U60: SY6280AAC, lcsc_footprints:C55136_SOT-23-5_L3.0-W1.7-P0.95-LS2.8-BL, symbol lcsc_imported:SY6280AAC_C55136
- R180, R187: value 1.65k -> 4.7k; KiLib_Generator (none) -> SMD_2terminal_chip_molded; LCSC C25869 -> C25900
Connections:
- net +5V: now also U59.5 (IN), U60.5 (IN)
- net +5V_BRIDGE: now also D22.1 (K), U60.1 (OUT)
- net +5V_MOD: now also U59.1 (OUT)
- net BRIDGE_PWR_EN: now also U60.4 (EN)
- net GND: now also D22.2 (A), R195.2, U59.2 (GND), U60.2 (GND); no longer R187.2
- net MOD_PWR_EN: now also U59.4 (EN)
- net BR_ILM: no longer names the net of R187.1
- net BR_ILM: now also U60.3 (ISET)
- net MOD_ILM: no longer names the net of R180.1
- net MOD_ILM: now also U59.3 (ISET)
- new net: R187.2, R195.1
Other:
- note added: "Link to the analog module: 24-pin 1.0 mm FFC (top and bottom contact). 1-3 +5V_MOD (U59 SY6280AAC power switch, ~1.45 A limit (4.7k), on at power-up; PD10 low = off) 4-6 GND, 7 DAC_SCLK, 8 DAC_DIN, 9 DAC_SYNC, 10 GND 11 ADC_SCLK, 12 ADC_SDO, 13 ADC_SDI, 14 GND, 15 ADC_CNVST, 16 GND 17 MOD_I2C_SDA (PF0), 18 MOD_I2C_SCL (PF1), own bus, 4.7k pull-ups, 19 GND, 20 MOD_RESET# (PD8), 21 MOD_PRESENT# (PD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"
- note removed: "Link to the analog module: 24-pin 1.0 mm FFC (top and bottom contact). 1-3 +5V_MOD (eFuse U59, ~1 A limit, on at power-up; PD10 low = off) 4-6 GND, 7 DAC_SCLK, 8 DAC_DIN, 9 DAC_SYNC, 10 GND 11 ADC_SCLK, 12 ADC_SDO, 13 ADC_SDI, 14 GND, 15 ADC_CNVST, 16 GND 17 MOD_I2C_SDA (PF0), 18 MOD_I2C_SCL (PF1), own bus, 4.7k pull-ups, 19 GND, 20 MOD_RESET# (PD8), 21 MOD_PRESENT# (PD9, module ties to GND) 22 G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"
