File: pcb/benchpod-digital/module-link.kicad_sch (KiCad schematic)
At the start: 21 parts, among them CN1 KH-FPC1.0-H2.0SMT-24P-QCHF, U59 SY6280AAC, U60 SY6280AAC

Commit message: drc fixes
Connections:
- net +5V_MOD: now also CN1.4
- net GND: no longer CN1.4
Changed lines of the file:
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@@
 	)
 	(label "+5V_MOD"
+		(at 195.58 82.55 180)
+		(effects
+			(font
+				(size 1.27 1.27)
+			)
+			(justify right bottom)
+		)
+	)
+	(label "+5V_MOD"
 		(at 195.58 74.93 180)
 		(effects
@@
 					(unit 1)
 				)
-			)
-		)
-	)
-	(symbol
-		(lib_id "power:GND")
-		(at 195.58 82.55 270)
-		(unit 1)
-		(body_style 1)
-		(exclude_from_sim no)
-		(in_bom yes)
-		(on_board yes)
-		(in_pos_files yes)
-		(dnp no)
-		(property "Reference" "#PWR0500"
-			(at 195.58 82.55 270)
-			(hide yes)
-			(show_name no)
-			(do_not_autoplace no)
-			(effects
-				(font
-					(size 1.27 1.27)
-				)
-			)
-		)
-		(property "Value" "GND"
-			(at 195.58 82.55 270)
-			(hide yes)
-			(show_name no)
-			(do_not_autoplace no)
-			(effects
-				(font
-					(size 1.27 1.27)
-				)
-			)
-		)
-		(property "Footprint" ""
-			(at 195.58 82.55 270)
-			(hide yes)
-			(show_name no)
-			(do_not_autoplace no)
-			(effects
-				(font
-					(size 1.27 1.27)
-				)
-			)
-		)
-		(property "Datasheet" ""
-			(at 195.58 82.55 270)
-			(hide yes)
-			(show_name no)
-			(do_not_autoplace no)
-			(effects
-				(font
-					(size 1.27 1.27)
-				)
-			)
-		)
-		(property "Description" "Power symbol creates a global label with name \"GND\" , ground"
-			(at 195.58 82.55 270)
-			(hide yes)
-			(show_name no)
-			(do_not_autoplace no)
-			(effects
-				(font
-					(size 1.27 1.27)
-				)
-			)
-		)
-		(pin "1"
-		)
-		(instances
-			(project "vbench-pod"
-				(path "/745fcf4b-2e0b-4fc4-95c0-f2e3fd40beb9/3b6fbda2-fc40-469d-a8f6-0fdb43fb58b6"
-					(reference "#PWR0500")
-					(unit 1)
-				)

Commit message: bom changes, cleanups
Parts:
- D22: value SMAJ5.0A_C2925443 -> SMAJ5.0A
Changed lines of the file:
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@@
 			)
 		)
-		(property "Value" "SMAJ5.0A_C2925443"
+		(property "Value" "SMAJ5.0A"
 			(at 116.84 173.99 0)
 			(show_name no)
