File: pcb/benchpod-digital/vbench-pod.kicad_pcb (KiCad board)
At the start: 4 copper layers, 98.5 x 118 mm, 322 parts, among them CN1 KH-FPC1.0-H2.0SMT-24P-QCHF, J1 X9555WR-2x13-6TV01, J10 Conn_02x02_Counter_Clockwise, J11 Conn_02x02_Counter_Clockwise, J4 DB2ERC-3.81-2P-BK, J5 DB2ERC-3.81-2P-BK, J6 DB2ERC-3.81-2P-BK, J7 HR911105A_C12074, SW1 TS24CA, SW2 TS24CA, U1 ICE40UP5K-SG48ITR, U10 TCAN1044VDRBRQ1, U18 SN74LVC2G66DCUR, U19 SN74LVC2G66DCUR, U2 W25Q64JVSSIQ, U20 SN74LVC2G66DCUR, U21 SN74LVC2G66DCUR, U22 SRV05-4.TCT, U23 SRV05-4.TCT, U24 SN74LVC2G66DCUR, U25 SRV05-4.TCT, U26 TPS259470ARPWR, U27 TPS259470ARPWR, U28 SRV05-4.TCT, U29 INA226AIDGSR, U30 TPS62130ARGTR, U31 AP2112K-1.2, U32 AP2112K-2.5TRG1, U33 INA226AIDGSR, U34 SRV05-4.TCT, U35 INA226AIDGSR, U5 STM32H563ZGT6, U52 AP2112K-1.8TRG1, U54 TCA9554PWR, U56 TCA9554PWR, U57 TPS259470ARPWR, U59 SY6280AAC, U6 LAN8742AI-CZ-TR, U60 SY6280AAC, U7 APS6404L-3SQR-SN, U8 TPS2116DRLR, X1 SX3M48.000B10F20TNN, Y1 6pF ±10ppm SMD2016-4P Crystal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, Y2 6pF ±10ppm SMD2016-4P Crystal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

Commit message: drc fixes
Routing:
- net /MOD_SPARE: track 9.59 -> 27.9 mm
- net +3V3: track 1038.4 -> 1027.7 mm, vias 92 -> 91
- net +5V_EFUSE: track 55.2 -> 50.5 mm, vias 6 -> 7
- net Net-(J4-Pin_1): track 129.3 -> 132.4 mm
- net +5V_IN: track 116.9 -> 115.6 mm, vias 8 -> 10
- net +5V: track 299.4 -> 300.7 mm
- net /Power/INA_IN_P2: track 33.0 -> 34.0 mm, vias 3 -> 4
- net LA_VCCIO: track 103.8 -> 103.2 mm
- net /MOD_PRESENT#: track 25.8 -> 25.3 mm
- net /MOD_DAC_SYNC: track 21.1 -> 20.6 mm
- net /MOD_DAC_SCLK: track 20.1 -> 19.6 mm
- net GND: track 309.7 -> 309.2 mm, vias 516 -> 554
- net /MOD_ADC_CNVST: track 2.95 -> 3.06 mm, vias 1 -> 0
- added copper zone on F.Cu, net +5V_EFUSE
- added copper zone on F.Cu, net +5V_IN
- added copper zone on F.Cu, net /Power/INA_IN_P2
- added copper zone on F.Cu, net Net-(J4-Pin_1)

Commit message: drc fixes - the end
Parts:
- added C10: 100n, Capacitor_SMD:C_0402_1005Metric, F.Cu at (106.0, 46.6)
- added C61: 1u, Capacitor_SMD:C_0402_1005Metric, F.Cu at (107.4, 46.5)
- moved R4 1.83 mm to (96.4, 54.6), turned to 90 degrees
- moved C11 0.18 mm to (105.3, 49.5)
Routing:
- net +3V3: track 1027.7 -> 1036.4 mm
- net /ICE_IO2: track 56.8 -> 52.3 mm
- net GND: track 309.2 -> 311.0 mm, vias 554 -> 556
- net +5V_EFUSE: track 50.5 -> 51.6 mm
- net /ICE_SCLK: track 63.4 -> 64.1 mm
- added copper zone on B.Cu, net /Power/INA_IN_P2
- added copper zone on B.Cu, net Net-(J4-Pin_1)

Commit message: drc fixes
Parts:
- added C67: 1u, Capacitor_SMD:C_0402_1005Metric, F.Cu at (102.3, 45.4)
- moved C19 1.63 mm to (93.6, 62.3)
- moved FB2 1.20 mm to (96.8, 58.1), turned to -90 degrees
- moved C55 1.02 mm to (96.7, 60.1), turned to 180 degrees
- moved R1 0.95 mm to (94.8, 60.1)
- moved R150 0.59 mm to (99.4, 62.3)
- moved C54 0.58 mm to (97.9, 61.9)
- moved Y2 0.48 mm to (100.2, 59.4)
- moved C50 0.48 mm to (101.3, 61.3)
- moved C51 0.46 mm to (99.3, 61.3)
- moved C34 0.39 mm to (96.9, 61.9)
Routing:
- net Net-(U5-VREF+): track 5.50 -> 8.10 mm
- net Net-(U5-VDDA): track 7.59 -> 9.87 mm
- net +3V3: track 1036.4 -> 1038.1 mm
- net LA_VCCIO: track 103.2 -> 104.2 mm
- net /NRST: track 116.3 -> 116.9 mm
- net /PH1: track 2.75 -> 2.16 mm
- net /PH0: track 6.84 -> 6.32 mm
- net GND: track 311.0 -> 311.2 mm, vias 556 -> 566
