File: pcb/benchpod-digital/vbench-pod.kicad_pcb (KiCad board)
At the start: 4 copper layers, 98.5 x 118 mm, 325 parts, among them CN1 KH-FPC1.0-H2.0SMT-24P-QCHF, J1 X9555WR-2x13-6TV01, J10 Conn_02x02_Counter_Clockwise, J11 Conn_02x02_Counter_Clockwise, J4 DB2ERC-3.81-2P-BK, J5 DB2ERC-3.81-2P-BK, J6 DB2ERC-3.81-2P-BK, J7 HR911105A_C12074, SW1 TS24CA, SW2 TS24CA, U1 ICE40UP5K-SG48ITR, U10 TCAN1044VDRBRQ1, U18 SN74LVC2G66DCUR, U19 SN74LVC2G66DCUR, U2 W25Q64JVSSIQ, U20 SN74LVC2G66DCUR, U21 SN74LVC2G66DCUR, U22 SRV05-4.TCT, U23 SRV05-4.TCT, U24 SN74LVC2G66DCUR, U25 SRV05-4.TCT, U26 TPS259470ARPWR, U27 TPS259470ARPWR, U28 SRV05-4.TCT, U29 INA226AIDGSR, U30 TPS62130ARGTR, U31 AP2112K-1.2, U32 AP2112K-2.5TRG1, U33 INA226AIDGSR, U34 SRV05-4.TCT, U35 INA226AIDGSR, U5 STM32H563ZGT6, U52 AP2112K-1.8TRG1, U54 TCA9554PWR, U56 TCA9554PWR, U57 TPS259470ARPWR, U59 SY6280AAC, U6 LAN8742AI-CZ-TR, U60 SY6280AAC, U7 APS6404L-3SQR-SN, U8 TPS2116DRLR, X1 SX3M48.000B10F20TNN, Y1 6pF ±10ppm SMD2016-4P Crystal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, Y2 6pF ±10ppm SMD2016-4P Crystal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

Commit message: drc fixes
Routing:
- net +3V3: track 1038.1 -> 1035.9 mm
- net /ICE_CRESET: track 33.6 -> 32.4 mm
- net /ICE_CDONE: track 32.5 -> 33.5 mm
- net /ICE_SPI_SI: track 53.6 -> 52.8 mm
- net GND: track 311.2 -> 311.3 mm, vias 566 -> 576

Commit message: drc fixes
Routing:
- net +3V3: track 1035.9 -> 1033.4 mm, vias 91 -> 89
- net GND: track 311.3 -> 310.9 mm, vias 576 -> 612
