File: pcb/benchpod-analog/analog-to-digital-v2.kicad_sch (KiCad schematic)
At the start: 48 parts, among them J10 BNC-KYWE-295-W4-N, J8 WJ15EDGRC-3.81-02P, K3 G6K-2F-Y DC5, K4 G6K-2F-Y DC5, U17 TMCP1A106MTRF, U36 MCP33131D-10-E/MS, U37 THS4551IRUNR, U40 OPA810IDBVR

Commit message: pcb work
Parts:
- removed TP4: TP ADC in, TestPoint:TestPoint_Pad_D1.5mm, symbol Connector:TestPoint
