File: pcb/benchpod-analog/analog-to-digital-v2.kicad_sch (KiCad schematic)
At the start: 47 parts, among them J10 BNC-KYWE-295-W4-N, J8 WJ15EDGRC-3.81-02P, K3 G6K-2F-Y DC5, K4 G6K-2F-Y DC5, U17 TMCP1A106MTRF, U36 MCP33131D-10-E/MS, U37 THS4551IRUNR, U40 OPA810IDBVR

Commit message: analog: black DORABO terminals, flush with the front panel
J8/J9 -> DB2ERC-3.81-2P-BK (C5259145, same as digital J4-J6), J11 -> DB2ERC-3.81-6P-BK
(C5244107, new footprint from EasyEDA + courtyard, no 3D model). Same pinout and pitch,
body centre x kept, pad row y 25.53 -> 24.271 (face 3.8 mm past the edge). Stale
C8465/WJ500V fields on J8/J9 corrected. Tracks to the old pads need rerouting.

Co-Authored-By: Claude Opus 5.5 <noreply@anthropic.com>
Parts:
- J8: value WJ15EDGRC-3.81-02P -> DB2ERC-3.81-2P-BK; footprint lcsc_footprints:C8387_CONN-TH_2P-P3.81_WJ15EDGRC-3.81-2P -> lcsc_footprints:C5259145_CONN-TH_2P-P3.81_DB2ERC-3.81-2P-BK; LCSC C8387 -> C5259145; LCSC Part C8465 -> C5259145; LCSC Part # C8465 -> C5259145; MFR. Part # WJ500V-5.08-2P -> DB2ERC-3.81-2P-BK; Manufacturer_Name (none) -> DORABO; Manufacturer_Part_Number (none) -> DB2ERC-3.81-2P-BK
Changed lines of the file:
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@@
 			)
 		)
-		(property "Value" "WJ15EDGRC-3.81-02P"
+		(property "Value" "DB2ERC-3.81-2P-BK"
 			(at 63.246 150.876 0)
 			(show_name no)
@@
 			)
 		)
-		(property "Footprint" "lcsc_footprints:C8387_CONN-TH_2P-P3.81_WJ15EDGRC-3.81-2P"
+		(property "Footprint" "lcsc_footprints:C5259145_CONN-TH_2P-P3.81_DB2ERC-3.81-2P-BK"
 			(at 53.34 154.94 0)
 			(hide yes)
@@
 			)
 		)
-		(property "Datasheet" "https://www.lcsc.com/datasheet/C8387.pdf"
+		(property "Datasheet" "https://www.lcsc.com/datasheet/C5259145.pdf"
 			(at 53.34 154.94 0)
 			(hide yes)
@@
 			)
 		)
-		(property "LCSC Part #" "C8465"
+		(property "LCSC Part #" "C5259145"
 			(at 53.34 154.94 0)
 			(hide yes)
@@
 			)
 		)
-		(property "MFR. Part #" "WJ500V-5.08-2P"
+		(property "MFR. Part #" "DB2ERC-3.81-2P-BK"
 			(at 53.34 154.94 0)
 			(hide yes)
@@
 			)
 		)
-		(property "LCSC" "C8387"
+		(property "LCSC" "C5259145"
 			(at 53.34 154.94 0)
 			(hide yes)
@@
 			)
 		)
-		(property "LCSC Part" "C8465"
+		(property "LCSC Part" "C5259145"
 			(at 53.34 154.94 0)
 			(hide yes)
@@
 			)
 		)
-		(property "Manufacturer_Name" ""
+		(property "Manufacturer_Name" "DORABO"
 			(at 53.34 154.94 0)
 			(hide yes)
@@
 			)
 		)
-		(property "Manufacturer_Part_Number" ""
+		(property "Manufacturer_Part_Number" "DB2ERC-3.81-2P-BK"
 			(at 53.34 154.94 0)
 			(hide yes)
