File: pcb/benchpod-analog/analog-to-digital-v2.kicad_sch (KiCad schematic)
At the start: 47 parts, among them J10 BNC-KYWE-295-W4-N, J8 DB2ERC-3.81-2P-BK, K3 G6K-2F-Y DC5, K4 G6K-2F-Y DC5, U17 TMCP1A106MTRF, U36 MCP33131D-10-E/MS, U37 THS4551IRUNR, U40 OPA810IDBVR

Commit message: analog module: ÷2 ADC low range (K5)
A second input range for small signals: ±5.46 V (÷2, 167 uV/count)
next to today's ±32.8 V (÷12), 6x the resolution on 0-5 V signals and on
the J8 current input (both share the divider).

- K5 (G6K-2F-Y DC5, same part as K3) driven by U53 OUT5 from U58 P5
  (R185 4.7k pull-down), LOW_RANGE_EN through the root sheet.
- Pole 1 swaps the bottom leg: R91 82.5k + C72 to GND (NC1, off) or
  R182 910k 0.1 % 25 ppm + C269 47 pF to GND (NO1, on). R90 stays in
  series, so 30 V into the D22 clamp is still ~33 uA.
- Pole 2 moves C271 (47 pF 100 V): to GND on the normal range (part of
  the bottom leg; C72 100 -> 51 pF keeps it at ~105 pF with strays), across
  R90 on the low range (top leg 56.4 pF). The open contacts never bridge
  the divider, so the normal range keeps the v3r3 compensation.
- C270 DNP pad for the first-article trim (adc_comp_sweep.py on both
  ranges); R183/R184 0 ohm DNP give the ÷12 divider without K5.
- ADC sheet A3 (like the power and DAC sheets) for room.

Netlist checked against the design; ERC adds only pin_to_pin notes from
the relay symbol's unspecified pin types (as K3/K4). PCB not updated.

Co-Authored-By: Claude Opus 5.5 <noreply@anthropic.com>
Parts:
- added C269, C270: 47p, Capacitor_SMD:C_0402_1005Metric, symbol Device:C
- added C271: 47p, Capacitor_SMD:C_0603_1608Metric, symbol Device:C
- added K5: G6K-2F-Y DC5, lcsc:RELAY-TH_G6K-2F-Y, symbol lcsc_lib:G6K-2F-YDC5
- added R182: 910k, Resistor_SMD:R_0603_1608Metric, symbol Device:R
- added R183, R184: 0, Resistor_SMD:R_0603_1608Metric, symbol Device:R
- C72: value 100p -> 51p; LCSC C327198 -> C541437
Connections:
- net +5V: now also K5.1
- net GND: now also K5.3, K5.7, R183.2, R184.2; no longer C72.2, R91.2
- net RELAY2_OUT: now also K5.5
- net ADC_DIV_MID: now reaches C140.2, C72.1, D22.3 (K/A), R90.2, R91.1, U40.3 (VIN+)
- net ADC_DIV_MID: now also C269.1, C270.1, C271.1, R182.1
- new net DIV_LEG_A: C72.2, K5.2, R183.1, R91.2
- new net DIV_LEG_B: C269.2, C270.2, K5.4, R182.2
- new net DIV_SW_C: C271.2, K5.6, R184.1
- new net LOW_RANGE_EN: K5.8
Other:
- note added: "ADC low range: K5, LOW_RANGE_EN (U53 OUT5, from U58 P5). K5 off = ±32.8 V (÷12, as v3r3). K5 on = ±5.46 V (÷2). Off: R91 + C72 51p + C271 47p to GND (NC1/NC2): 82.5k || ~105 pF (98p + ~7p stray), top 9.1p + 0.3p. On: R182 910k || C269 47p to GND (NO1), C271 across R90 (NO2): top 9.1 + 47 + 0.3 = 56.4p, bottom 47p + ~8p stray. Low range input 1.82 Mohm: 1x leads, not 10x probes. Final C269/C271 (C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"
