File: pcb/benchpod-analog/analog-to-digital-v2.kicad_sch (KiCad schematic)
At the start: 54 parts, among them J10 BNC-KYWE-295-W4-N, J8 DB2ERC-3.81-2P-BK, K3 G6K-2F-Y DC5, K4 G6K-2F-Y DC5, K5 G6K-2F-Y DC5, U17 TMCP1A106MTRF, U36 MCP33131D-10-E/MS, U37 THS4551IRUNR, U40 OPA810IDBVR

Commit message: K5 routing
Parts:
- added C234: 1u, Capacitor_SMD:C_0402_1005Metric, symbol Device:C
- added C235: 100n, Capacitor_SMD:C_0402_1005Metric, symbol Device:C
Connections:
- net +5V: now also C234.2, C235.2
- net GND: now also C234.1, C235.1
Other:
- moved on the sheet: K5, R183, R184
