File: pcb/benchpod-analog/digital-to-analog-v2.kicad_sch (KiCad schematic)
At the start: 65 parts, among them J11 WJ15EDGRC-3.81-06P, J9 WJ15EDGRC-3.81-02P, K1 G6K-2F-Y DC5, K2 G6K-2F-Y DC5, Q1 BCP56, U43 DAC8554IPWR, U44 OPA2365AIDR, U45 OPA2992IDR, U51 OPA2992IDR, U9 XTR116UA/2K5

Commit message: pcb work
Parts:
- removed TP1: TP 0-3.3V, TestPoint:TestPoint_Pad_D1.5mm, symbol Connector:TestPoint
- removed TP2: TP 0-5V, TestPoint:TestPoint_Pad_D1.5mm, symbol Connector:TestPoint
- removed TP3: TP +-12V, TestPoint:TestPoint_Pad_D1.5mm, symbol Connector:TestPoint
