File: pcb/benchpod-analog/digital-to-analog-v2.kicad_sch (KiCad schematic)
At the start: 62 parts, among them J11 WJ15EDGRC-3.81-06P, J9 WJ15EDGRC-3.81-02P, K1 G6K-2F-Y DC5, K2 G6K-2F-Y DC5, Q1 BCP56, U43 DAC8554IPWR, U44 OPA2365AIDR, U45 OPA2992IDR, U51 OPA2992IDR, U9 XTR116UA/2K5

Commit message: analog: black DORABO terminals, flush with the front panel
J8/J9 -> DB2ERC-3.81-2P-BK (C5259145, same as digital J4-J6), J11 -> DB2ERC-3.81-6P-BK
(C5244107, new footprint from EasyEDA + courtyard, no 3D model). Same pinout and pitch,
body centre x kept, pad row y 25.53 -> 24.271 (face 3.8 mm past the edge). Stale
C8465/WJ500V fields on J8/J9 corrected. Tracks to the old pads need rerouting.

Co-Authored-By: Claude Opus 5.5 <noreply@anthropic.com>
Parts:
- J11: value WJ15EDGRC-3.81-06P -> DB2ERC-3.81-6P-BK; footprint lcsc_footprints:C7246_CONN-TH_WJ15EDGRC-3.81-6P -> lcsc_footprints:C5244107_HDR-TH_DB2ERC-3.81-6P-BK; LCSC C7246 -> C5244107
- J9: value WJ15EDGRC-3.81-02P -> DB2ERC-3.81-2P-BK; footprint lcsc_footprints:C8387_CONN-TH_2P-P3.81_WJ15EDGRC-3.81-2P -> lcsc_footprints:C5259145_CONN-TH_2P-P3.81_DB2ERC-3.81-2P-BK; LCSC C8387 -> C5259145; LCSC Part C8465 -> C5259145; LCSC Part # C8465 -> C5259145; MFR. Part # WJ500V-5.08-2P -> DB2ERC-3.81-2P-BK; Manufacturer_Name (none) -> DORABO; Manufacturer_Part_Number (none) -> DB2ERC-3.81-2P-BK
Changed lines of the file:
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@@
 			)
 		)
-		(property "Value" "WJ15EDGRC-3.81-02P"
+		(property "Value" "DB2ERC-3.81-2P-BK"
 			(at 116.332 246.126 0)
 			(show_name no)
@@
 			)
 		)
-		(property "Footprint" "lcsc_footprints:C8387_CONN-TH_2P-P3.81_WJ15EDGRC-3.81-2P"
-			(at 133.35 240.03 0)
-			(hide yes)
-			(show_name no)
-			(do_not_autoplace no)
-			(effects
-				(font
-					(size 1.27 1.27)
-				)
-			)
-		)
-		(property "Datasheet" "https://www.lcsc.com/datasheet/C8387.pdf"
+		(property "Footprint" "lcsc_footprints:C5259145_CONN-TH_2P-P3.81_DB2ERC-3.81-2P-BK"
+			(at 133.35 240.03 0)
+			(hide yes)
+			(show_name no)
+			(do_not_autoplace no)
+			(effects
+				(font
+					(size 1.27 1.27)
+				)
+			)
+		)
+		(property "Datasheet" "https://www.lcsc.com/datasheet/C5259145.pdf"
 			(at 133.35 240.03 0)
 			(hide yes)
@@
 			)
 		)
-		(property "LCSC Part #" "C8465"
-			(at 133.35 240.03 0)
-			(hide yes)
-			(show_name no)
-			(do_not_autoplace no)
-			(effects
-				(font
-					(size 1.27 1.27)
-				)
-			)
-		)
-		(property "MFR. Part #" "WJ500V-5.08-2P"
-			(at 133.35 240.03 0)
-			(hide yes)
-			(show_name no)
-			(do_not_autoplace no)
-			(effects
-				(font
-					(size 1.27 1.27)
-				)
-			)
-		)
-		(property "LCSC" "C8387"
-			(at 133.35 240.03 0)
-			(hide yes)
-			(show_name no)
-			(do_not_autoplace no)
-			(effects
-				(font
-					(size 1.27 1.27)
-				)
-			)
-		)
-		(property "LCSC Part" "C8465"
+		(property "LCSC Part #" "C5259145"
+			(at 133.35 240.03 0)
+			(hide yes)
+			(show_name no)
+			(do_not_autoplace no)
+			(effects
+				(font
+					(size 1.27 1.27)
+				)
+			)
+		)
+		(property "MFR. Part #" "DB2ERC-3.81-2P-BK"
+			(at 133.35 240.03 0)
+			(hide yes)
+			(show_name no)
+			(do_not_autoplace no)
+			(effects
+				(font
+					(size 1.27 1.27)
+				)
+			)
+		)
+		(property "LCSC" "C5259145"
+			(at 133.35 240.03 0)
+			(hide yes)
+			(show_name no)
+			(do_not_autoplace no)
+			(effects
+				(font
+					(size 1.27 1.27)
+				)
+			)
+		)
+		(property "LCSC Part" "C5259145"
 			(at 133.35 240.03 0)
 			(hide yes)
@@
 			)
 		)
-		(property "Manufacturer_Name" ""
-			(at 133.35 240.03 0)
-			(hide yes)
-			(show_name no)
-			(do_not_autoplace no)
-			(effects
-				(font
-					(size 1.27 1.27)
-				)
-			)
-		)
-		(property "Manufacturer_Part_Number" ""
+		(property "Manufacturer_Name" "DORABO"
+			(at 133.35 240.03 0)
+			(hide yes)
+			(show_name no)
+			(do_not_autoplace no)
+			(effects
+				(font
+					(size 1.27 1.27)
+				)
+			)
+		)
+		(property "Manufacturer_Part_Number" "DB2ERC-3.81-2P-BK"
 			(at 133.35 240.03 0)
 			(hide yes)
@@
 			)
 		)
-		(property "Value" "WJ15EDGRC-3.81-06P"
+		(property "Value" "DB2ERC-3.81-6P-BK"
 			(at 322.58 74.93 0)
 			(show_name no)
@@
 			)
 		)
-		(property "Footprint" "lcsc_footprints:C7246_CONN-TH_WJ15EDGRC-3.81-6P"
+		(property "Footprint" "lcsc_footprints:C5244107_HDR-TH_DB2ERC-3.81-6P-BK"
 			(at 320.04 62.23 0)
 			(hide yes)
@@
 			)
 		)
-		(property "Datasheet" "https://www.lcsc.com/datasheet/C7246.pdf"
+		(property "Datasheet" "https://www.lcsc.com/datasheet/C5244107.pdf"
 			(at 320.04 62.23 0)
 			(hide yes)
@@
 			)
 		)
-		(property "Description" "DAC outputs: 1 0-3.3V, 3 0-5V, 5 +-12V, 2/4/6 GND (3.81 mm pluggable, green)"
+		(property "Description" "DAC outputs: 1 0-3.3V, 3 0-5V, 5 +-12V, 2/4/6 GND (3.81 mm pluggable, black)"
 			(at 320.04 62.23 0)
 			(hide yes)
@@
 			)
 		)
-		(property "LCSC" "C7246"
+		(property "LCSC" "C5244107"
 			(at 320.04 62.23 0)
 			(hide yes)
