File: pcb/benchpod-analog/digital-to-analog-v2.kicad_sch (KiCad schematic)
At the start: 62 parts, among them J11 DB2ERC-3.81-6P-BK, J9 DB2ERC-3.81-2P-BK, K1 G6K-2F-Y DC5, K2 G6K-2F-Y DC5, Q1 BCP56, U43 DAC8554IPWR, U44 OPA2365AIDR, U45 OPA2992IDR, U51 OPA2992IDR, U9 XTR116UA/2K5

Commit message: pcb work
Parts:
- added C216: 100n, Capacitor_SMD:C_0402_1005Metric, symbol Device:C
Connections:
- net +3V3A: now also C216.2
- net GND: now also C216.1

Commit message: vias, fixes
Changed lines of the file:
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@@
 	)
 	(label "BUFFER_VMID"
-		(at 218.44 173.99 0)
+		(at 218.44 173.99 180)
 		(effects
 			(font
 				(size 1.27 1.27)
 			)
-			(justify left bottom)
+			(justify right bottom)
 		)
 	)
