File: pcb/benchpod-analog/digital-to-analog-v2.kicad_sch (KiCad schematic)
At the start: 63 parts, among them J11 DB2ERC-3.81-6P-BK, J9 DB2ERC-3.81-2P-BK, K1 G6K-2F-Y DC5, K2 G6K-2F-Y DC5, Q1 BCP56, U43 DAC8554IPWR, U44 OPA2365AIDR, U45 OPA2992IDR, U51 OPA2992IDR, U9 XTR116UA/2K5

Commit message: analog module: use reserved JLC stock for C207/C208 and U42
C207/C208 5.1 pF: C2297586 (11 left at JLC) -> C20617868 (FH 0603 C0G 50 V,
100 reserved); op-amp feedback caps, 50 V is plenty. C140 9.1 pF 250 V stays.
U42 LM7705MM/NOPB C129980 -> LM7705MMX/NOPB C2070761 (same chip and
VSSOP-8 package, larger reel; 10 reserved). Schematic and board fields both.

Co-Authored-By: Claude Opus 5.5 <noreply@anthropic.com>
Parts:
- C207, C208: LCSC C2297586 -> C20617868
Changed lines of the file:
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@@
 			)
 		)
-		(property "LCSC" "C2297586"
+		(property "LCSC" "C20617868"
 			(at 250.19 198.12 90)
 			(hide yes)
@@
 			)
 		)
-		(property "LCSC" "C2297586"
+		(property "LCSC" "C20617868"
 			(at 242.57 162.56 90)
 			(hide yes)
