File: pcb/benchpod-analog/vbench-pod.kicad_pcb (KiCad board)
At the start: 4 copper layers, 98.9 x 118.2 mm, 247 parts, among them CN1 KH-FPC1.0-H2.0SMT-24P-QCHF, J8 Screw_Terminal_01x02, J9 Screw_Terminal_01x02, K1 G6K-2F-Y DC5, K2 G6K-2F-Y DC5, K3 G6K-2F-Y DC5, K4 G6K-2F-Y DC5, Q1 BCP56, U11 HX PZ2.54-1X2P ZZ, U12 HX PZ2.54-1X2P ZZ, U13 HX PZ2.54-1X2P ZZ, U14 HX PZ2.54-1X2P ZZ, U15 TPS7A2045PDBVR, U16 TLV61046ADBVR, U17 TMCP1A106MTRF, U3 TPS7A2050PDQNR, U30 AP2112K-3.3, U36 MCP33131D-10-E/MS, U37 THS4551IRUNR, U38 ADR4540BRZ-R7, U39 AP2112K-1.8TRG1, U40 OPA810IDBVR, U41 LM27761DSGR, U42 LM7705MM/NOPB, U43 DAC8554IPWR, U44 OPA2365AIDR, U45 OPA2992IDR, U46 AP2112K-3.3, U49 TPS65131RGER, U50 TPS7A1901DRBR, U51 OPA2992IDR, U53 TPL7407LAPWR, U58 TCA9554PWR, U61 24C32, U9 XTR116UA/2K5

Commit message: pcb work
Parts:
- removed D7, D8: SMAJ36CA, lcsc:SMA_L4.3-W2.6-LS5.0-BI
- removed R165, R166, R167, R20: 0, Resistor_SMD:R_0402_1005Metric
- removed RF1, RF2, RF3, RF4: HC-SMA-KWE-14.5H-D002-01, lcsc:SMA-TH_BWSMA-KWE-Z001
- removed U11, U12, U13, U14: HX PZ2.54-1X2P ZZ, lcsc_footprints:C32713268_HDR-TH_2P-P2_54-V-M-3
- added D22: BAV199, lcsc_footprints:C145516_SOT-23_L2.9-W1.3-P1.90-LS2.4-BR, F.Cu at (70.3, 44.6)
- added J10: BNC-KYWE-295-W4-N, lcsc_footprints:C41416668_BNC-TH_BNC-KYWE-295-W4-N, F.Cu at (53.9, 26.4)
- added J11: WJ15EDGRC-3.81-06P, lcsc_footprints:C7246_CONN-TH_WJ15EDGRC-3.81-6P, F.Cu at (114.4, 27.8)
- J8, J9: value Screw_Terminal_01x02 -> WJ15EDGRC-3.81-02P; footprint lcsc:CONN-TH_2P-P5.00_WJ500V-5.08-2P -> lcsc_footprints:C8387_CONN-TH_2P-P3.81_WJ15EDGRC-3.81-2P
- R90: footprint Resistor_SMD:R_0603_1608Metric -> Resistor_SMD:R_1206_3216Metric
- moved C246 56.3 mm to (67.9, 127.9), turned to 90 degrees
- moved C247 56.1 mm to (65.5, 124.8), turned to 180 degrees
- moved C248 55.2 mm to (65.5, 123.7), turned to 180 degrees
- moved C193 53.7 mm to (69.9, 127.2), turned to 180 degrees
- moved U3 53.5 mm to (65.8, 121.9), turned to -90 degrees
- moved C194 52.7 mm to (69.9, 126.2), turned to 180 degrees
- moved C249 52.5 mm to (65.8, 120.6), turned to 0 degrees
- moved C252 51.6 mm to (65.8, 119.5), turned to 0 degrees
- moved U50 51.1 mm to (69.0, 123.6), turned to 180 degrees
- moved C250 50.6 mm to (65.8, 117.9), turned to 180 degrees
- moved C265 50.4 mm to (72.7, 126.8), turned to 180 degrees
- moved C158 49.7 mm to (72.4, 125.8), turned to 0 degrees
- moved R121 49.4 mm to (68.3, 120.5), turned to -90 degrees
- moved C159 48.7 mm to (72.4, 124.8), turned to 0 degrees
- moved D9 48.5 mm to (81.3, 25.0)
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Connections:
- net Net-(D17-AK) renamed /digital to analog v2/OUT_3V3
- net Net-(D20-A1) renamed /digital to analog v2/OUT_12V
Routing:
- net +3V3A: track 131.6 -> 44.7 mm, vias 4 -> 3
- net /analog to digital v2/AMP_MEASURE_IN: track 68.5 -> 7.00 mm
- net 5VA: track 140.3 -> 92.2 mm, vias 12 -> 8
- net -5VA: track 76.4 -> 33.4 mm, vias 2 -> 1
- net /AMP_MEAS_EN: track 86.2 -> 44.1 mm, vias 2 -> 1
- net /DAC_TO_ADC: track 52.0 -> 14.0 mm, vias 4 -> 0
- net /CAL_PATH_EN: track 74.5 -> 44.8 mm, vias 2 -> 1
- net −0V232: track 73.8 -> 46.1 mm, vias 8 -> 5
- net +5V: track 258.4 -> 231.2 mm, vias 19 -> 17
- net -14V_ANA: track 89.8 -> 67.8 mm
- net /analog to digital v2/RELAY1_IN: track 28.0 -> 7.00 mm
- net /digital to analog v2/OUT_12V: track 34.8 -> 14.0 mm
- net +1V8A: track 62.6 -> 47.0 mm
- net +5V5_ANA: track 117.5 -> 102.8 mm, vias 12 -> 11
- net Net-(D9-A): track 22.2 -> 7.97 mm
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- added copper zone on F.Cu, net +5V
Other:
- board text removed: "-+12V DAC"
- board text removed: "0-3V3 DAC"
- board text removed: "0-5V DAC"

Commit message: placement
Parts:
- moved Q1 43.8 mm to (84.1, 36.4), turned to 0 degrees
- moved C243 42.5 mm to (81.0, 39.0), turned to 180 degrees
- moved C215 41.0 mm to (80.9, 40.3), turned to 0 degrees
- moved C241 38.8 mm to (84.0, 40.3), turned to 0 degrees
- moved C242 37.2 mm to (86.7, 40.3), turned to 180 degrees
- moved U9 34.5 mm to (84.0, 44.9), turned to -90 degrees
- moved R162 33.5 mm to (80.8, 48.4), turned to 0 degrees
- moved C244 31.7 mm to (88.4, 44.8), turned to 90 degrees
- moved R82 29.5 mm to (84.2, 49.2), turned to 90 degrees
- moved C208 26.8 mm to (94.7, 42.4)
- moved C214 26.8 mm to (107.3, 34.0)
- moved K2 26.8 mm to (103.6, 39.7)
- moved R126 26.8 mm to (94.6, 31.4)
- moved R127 26.8 mm to (95.1, 33.0)
- moved R128 26.8 mm to (109.6, 37.6)
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Routing:
- net AREF_4V096: track 121.0 -> 0.00 mm, vias 10 -> 0
- net +3V3: track 92.7 -> 0.00 mm, vias 9 -> 0
- net GND: track 192.1 -> 100.8 mm, vias 283 -> 141
- net +5V: track 231.2 -> 144.6 mm, vias 17 -> 7
- net /ANA14_EN: track 99.6 -> 18.9 mm, vias 4 -> 1
- net 5VA: track 92.2 -> 31.1 mm, vias 8 -> 4
- net +4V5_DAC: track 64.7 -> 4.85 mm, vias 3 -> 0
- net +5V5_ANA: track 102.8 -> 43.0 mm, vias 11 -> 3
- net /digital to analog v2/TO_12V: track 52.0 -> 0.00 mm
- net /CAL_PATH_EN: track 44.8 -> 0.00 mm, vias 1 -> 0
- net /AMP_MEAS_EN: track 44.1 -> 0.00 mm, vias 1 -> 0
- net /CAL1_EN: track 34.8 -> 0.00 mm, vias 2 -> 0
- net Net-(D9-K): track 26.8 -> 0.00 mm
- net Net-(U51C--INB): track 26.2 -> 0.00 mm
- net /CAL2_EN: track 23.5 -> 0.00 mm, vias 2 -> 0
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