File: pcb/benchpod-analog/vbench-pod.kicad_pcb (KiCad board)
At the start: 4 copper layers, 98.5 x 120.2 mm, 236 parts, among them CN1 KH-FPC1.0-H2.0SMT-24P-QCHF, J10 BNC-KYWE-295-W4-N, J11 WJ15EDGRC-3.81-06P, J8 WJ15EDGRC-3.81-02P, J9 WJ15EDGRC-3.81-02P, K1 G6K-2F-Y DC5, K2 G6K-2F-Y DC5, K3 G6K-2F-Y DC5, K4 G6K-2F-Y DC5, Q1 BCP56, U15 TPS7A2045PDBVR, U16 TLV61046ADBVR, U17 TMCP1A106MTRF, U3 TPS7A2050PDQNR, U30 AP2112K-3.3, U36 MCP33131D-10-E/MS, U37 THS4551IRUNR, U38 ADR4540BRZ-R7, U39 AP2112K-1.8TRG1, U40 OPA810IDBVR, U41 LM27761DSGR, U42 LM7705MM/NOPB, U43 DAC8554IPWR, U44 OPA2365AIDR, U45 OPA2992IDR, U46 AP2112K-3.3, U49 TPS65131RGER, U50 TPS7A1901DRBR, U51 OPA2992IDR, U53 TPL7407LAPWR, U58 TCA9554PWR, U61 24C32, U9 XTR116UA/2K5

Commit message: pcb alignment work
Parts:
- moved C268 30.2 mm to (108.7, 67.2), turned to 90 degrees
- moved C107 29.4 mm to (122.2, 70.4)
- moved C109 29.4 mm to (123.2, 70.4)
- moved C110 29.4 mm to (122.2, 73.3)
- moved C114 29.4 mm to (123.3, 73.3)
- moved C106 29.4 mm to (120.8, 69.8)
- moved U30 25.1 mm to (127.3, 71.1)
- moved U61 23.6 mm to (111.8, 71.7), turned to 90 degrees
- moved C175 21.3 mm to (108.4, 92.4)
- moved C178 21.3 mm to (108.7, 97.8)
- moved C180 21.3 mm to (111.0, 97.3)
- moved C181 21.3 mm to (121.2, 88.7)
- moved C183 21.3 mm to (113.1, 92.5)
- moved C184 21.3 mm to (117.3, 93.6)
- moved C185 21.3 mm to (114.2, 92.2)
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Routing:
- net /ADC_CNVST: track 0.00 -> 27.4 mm
- net /ADC_SDO: track 0.00 -> 24.9 mm
- net /ADC_SCLK: track 0.00 -> 23.6 mm
- net GND: track 100.8 -> 123.2 mm, vias 141 -> 169
- net /ADC_SDI: track 0.00 -> 22.1 mm
- net /analog to digital v2/RELAY2_IN: track 7.00 -> 21.8 mm
- net +14V_ANA: track 36.1 -> 24.1 mm
- net 5VA: track 31.1 -> 42.4 mm, vias 4 -> 6
- net Net-(U36-AIN-): track 0.00 -> 11.0 mm
- net Net-(D22-K/A): track 0.00 -> 10.6 mm
- net -5VA: track 33.4 -> 43.8 mm, vias 1 -> 3
- net Net-(U36-AIN+): track 0.00 -> 8.68 mm
- net /analog to digital v2/RELAY1_IN: track 7.00 -> 15.6 mm
- net 2.05V: track 0.00 -> 7.41 mm, vias 0 -> 2
- net Net-(U40-VIN-): track 0.00 -> 7.04 mm
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- added copper zone on In1.Cu, net (none)
- added copper zone on In2.Cu, net (none)
- added copper zone on F.Cu, net GND
