File: pcb/benchpod-analog/vbench-pod.kicad_pcb (KiCad board)
At the start: 4 copper layers, 98.5 x 120.2 mm, 236 parts, among them CN1 KH-FPC1.0-H2.0SMT-24P-QCHF, J10 BNC-KYWE-295-W4-N, J11 DB2ERC-3.81-6P-BK, J8 DB2ERC-3.81-2P-BK, J9 DB2ERC-3.81-2P-BK, K1 G6K-2F-Y DC5, K2 G6K-2F-Y DC5, K3 G6K-2F-Y DC5, K4 G6K-2F-Y DC5, Q1 BCP56, U15 TPS7A2045PDBVR, U16 TLV61046ADBVR, U17 TMCP1A106MTRF, U3 TPS7A2050PDQNR, U30 AP2112K-3.3, U36 MCP33131D-10-E/MS, U37 THS4551IRUNR, U38 ADR4540BRZ-R7, U39 AP2112K-1.8TRG1, U40 OPA810IDBVR, U41 LM27761DSGR, U42 LM7705MM/NOPB, U43 DAC8554IPWR, U44 OPA2365AIDR, U45 OPA2992IDR, U46 AP2112K-3.3, U49 TPS65131RGER, U50 TPS7A1901DRBR, U51 OPA2992IDR, U53 TPL7407LAPWR, U58 TCA9554PWR, U61 24C32, U9 XTR116UA/2K5

Commit message: pcb work
Parts:
- moved C158 65.5 mm to (131.3, 76.4), turned to 180 degrees
- moved C159 64.3 mm to (131.2, 77.4), turned to 180 degrees
- moved FB11 59.4 mm to (127.5, 76.6), turned to 0 degrees
- moved U42 57.5 mm to (128.4, 79.3), turned to 90 degrees
- moved C153 54.6 mm to (128.5, 82.1), turned to 180 degrees
- moved C224 52.9 mm to (124.8, 78.4), turned to -90 degrees
- moved C251 48.6 mm to (122.1, 94.6), turned to 180 degrees
- moved C193 48.3 mm to (122.1, 101.9)
- moved C194 48.3 mm to (122.1, 100.9)
- moved C195 48.3 mm to (123.3, 97.6)
- moved C198 48.3 mm to (122.1, 95.6)
- moved R121 48.3 mm to (120.5, 95.2)
- moved U50 48.3 mm to (121.3, 98.3)
- moved C157 47.7 mm to (123.2, 77.9)
- moved C173 47.6 mm to (119.3, 77.6), turned to 0 degrees
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Routing:
- net +5V: track 150.7 -> 84.6 mm
- net -14V_ANA: track 62.1 -> 20.4 mm, vias 3 -> 1
- net +5V5_ANA: track 43.0 -> 6.53 mm, vias 3 -> 1
- net +1V8A: track 42.7 -> 6.97 mm, vias 3 -> 1
- net −0V232: track 36.3 -> 3.17 mm, vias 4 -> 0
- net Net-(J9-Pin_2): track 0.00 -> 32.4 mm
- net Net-(D9-K): track 0.00 -> 29.8 mm
- net +3V3A: track 44.7 -> 72.9 mm, vias 3 -> 4
- net -5VA: track 43.8 -> 15.9 mm, vias 3 -> 2
- net 5VA: track 42.4 -> 26.1 mm, vias 6 -> 4
- net Net-(Q1-E): track 0.00 -> 15.8 mm
- net +6V_ANA: track 22.7 -> 7.11 mm, vias 2 -> 0
- net GND: track 123.2 -> 110.4 mm, vias 168 -> 142
- net Net-(U9-IIN): track 0.00 -> 9.58 mm
- net Net-(U50-EN): track 14.8 -> 5.28 mm
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
Commit message: pcb work
Parts:
- added C216: 100n, Capacitor_SMD:C_0402_1005Metric, F.Cu at (122.6, 30.0)
- moved U53 24.4 mm to (86.5, 69.3)
- moved U58 24.4 mm to (99.8, 69.4)
- moved C211 24.4 mm to (88.1, 64.8)
- moved R161 24.4 mm to (99.6, 64.3)
- moved R170 24.4 mm to (95.3, 73.7)
- moved C227 24.4 mm to (96.8, 67.8)
- moved C229 24.4 mm to (96.8, 65.9)
- moved R171 24.4 mm to (98.7, 74.4)
- moved R172 24.4 mm to (100.8, 74.4)
- moved R173 24.4 mm to (96.5, 71.6)
- moved C210 24.4 mm to (92.6, 75.7)
- moved C126 17.3 mm to (80.9, 78.6)
- moved C128 17.3 mm to (82.0, 78.6)
- moved U38 17.3 mm to (86.3, 79.8)
- moved C130 17.3 mm to (91.7, 79.9)
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Routing:
- net /digital to analog v2/TO_5V: track 0.00 -> 46.7 mm
- net /digital to analog v2/TO_3V3: track 0.00 -> 41.2 mm
- net /DAC_DIN: track 25.5 -> 52.5 mm
- net /DAC_SCLK: track 19.9 -> 46.9 mm
- net /I2C0_SDA: track 51.0 -> 25.0 mm
- net /I2C0_SCL: track 51.0 -> 25.1 mm
- net GND: track 110.4 -> 134.8 mm, vias 142 -> 166
- net +5V5_ANA: track 6.53 -> 30.3 mm, vias 1 -> 5
- net Net-(D19-A1): track 0.00 -> 21.8 mm
- net /CAL1_EN: track 0.00 -> 20.5 mm, vias 0 -> 1
- net /digital to analog v2/OUT_12V: track 0.00 -> 19.0 mm
- net /digital to analog v2/TO_5V_SMA: track 0.00 -> 17.9 mm
- net /digital to analog v2/TO_12V: track 0.00 -> 17.4 mm
- net Net-(U45C-OUTB): track 0.00 -> 15.4 mm
- net /DAC_TO_ADC: track 7.00 -> 21.0 mm
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
Commit message: pcb work
Parts:
- moved C126 26.2 mm to (105.7, 87.0), turned to 90 degrees
- moved FB9 25.0 mm to (105.7, 84.7), turned to -90 degrees
- moved C128 24.1 mm to (104.6, 87.0), turned to 90 degrees
- moved U38 15.2 mm to (100.3, 85.8), turned to 90 degrees
- moved D16 10.9 mm to (91.9, 118.1), turned to 0 degrees
- moved R172 10.8 mm to (90.4, 77.5), turned to -90 degrees
- moved R171 9.80 mm to (89.4, 77.5), turned to -90 degrees
- moved C210 9.45 mm to (92.4, 66.2)
- moved R161 9.30 mm to (105.4, 71.6), turned to 180 degrees
- moved C114 8.88 mm to (121.1, 64.7), turned to -90 degrees
- moved C110 8.88 mm to (120.1, 64.7), turned to -90 degrees
- moved C169 8.43 mm to (131.7, 33.9)
- moved R170 7.92 mm to (88.4, 77.5), turned to -90 degrees
- moved C132 7.87 mm to (95.9, 85.7), turned to 90 degrees
- moved R173 7.75 mm to (91.4, 77.5)
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Routing:
- net +5V: track 90.1 -> 339.4 mm, vias 7 -> 14
- net AREF_4V096: track 12.4 -> 148.0 mm, vias 0 -> 5
- net /CAL_PATH_EN: track 0.00 -> 73.3 mm, vias 0 -> 4
- net /DAC_TO_ADC: track 21.0 -> 84.1 mm, vias 0 -> 2
- net /AMP_MEAS_EN: track 0.00 -> 51.2 mm, vias 0 -> 4
- net /CAL2_EN: track 0.00 -> 36.6 mm, vias 0 -> 2
- net /digital to analog v2/BUFFER_VMID: track 1.37 -> 29.9 mm, vias 0 -> 2
- net /CAL1_EN: track 20.5 -> 46.9 mm, vias 1 -> 2
- net /analog to digital v2/AMP_MEASURE_IN: track 7.00 -> 25.8 mm
- net /ANA14_EN: track 18.9 -> 5.60 mm
- net /analog switching/CAL1: track 0.00 -> 12.8 mm
- net /analog switching/CAL2: track 0.00 -> 12.0 mm
- net /analog switching/AMP_MEASURE: track 0.00 -> 11.3 mm
- net /digital to analog v2/DAC_OUTPUT: track 0.00 -> 11.0 mm
- net /analog switching/CAL_PATH: track 0.00 -> 10.7 mm
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- added copper zone on F.Cu, net /Analog Power v2/INP
- added copper zone on F.Cu, net Net-(C175-Pad2)

Commit message: pcb work - all connected
Parts:
- moved C153 64.0 mm to (67.8, 62.1), turned to 90 degrees
- moved C154 61.1 mm to (68.0, 57.7), turned to 180 degrees
- moved U42 60.4 mm to (70.5, 62.0), turned to 0 degrees
- moved C159 60.1 mm to (72.4, 64.8), turned to 90 degrees
- moved C158 58.9 mm to (73.5, 64.8), turned to 90 degrees
- moved C224 57.0 mm to (71.5, 58.3), turned to 180 degrees
- moved FB11 56.5 mm to (73.2, 61.1), turned to -90 degrees
- moved C157 55.5 mm to (71.9, 56.7), turned to 0 degrees
- moved C261 32.3 mm to (117.3, 117.3)
- moved C262 32.3 mm to (117.0, 118.7)
- moved C264 32.3 mm to (116.6, 114.8)
- moved FB8 32.3 mm to (117.0, 111.6)
- moved L1 32.3 mm to (121.0, 119.9)
- moved R180 32.3 mm to (119.0, 113.0)
- moved U16 32.3 mm to (119.0, 115.3)
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Routing:
- net +3V3: track 4.78 -> 165.7 mm, vias 0 -> 7
- net 5VA: track 27.2 -> 181.2 mm, vias 6 -> 8
- net -14V_ANA: track 18.9 -> 132.2 mm, vias 1 -> 2
- net +5V5_ANA: track 31.8 -> 119.2 mm
- net +14V_ANA: track 20.7 -> 96.0 mm
- net /ANA14_EN: track 5.60 -> 73.2 mm, vias 1 -> 0
- net +4V5_DAC: track 2.05 -> 63.0 mm, vias 1 -> 2
- net +3V3A: track 74.0 -> 131.5 mm, vias 4 -> 6
- net -5VA: track 15.9 -> 69.7 mm, vias 2 -> 4
- net +1V8A: track 6.97 -> 58.7 mm, vias 1 -> 2
- net +5V: track 339.4 -> 380.3 mm
- net /I2C0_SCL: track 25.1 -> 57.6 mm
- net /I2C0_SDA: track 25.0 -> 57.2 mm
- net GND: track 142.5 -> 167.9 mm, vias 192 -> 224
- net −0V232: track 4.36 -> 14.0 mm
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- added copper zone on F.Cu, net Net-(D15-K)

Commit message: pcb work - pours
Routing:
- net GND: track 167.9 -> 164.9 mm, vias 224 -> 250
- net /analog switching/CAL_PATH: track 10.7 -> 9.38 mm
- net Net-(D19-A1): track 22.9 -> 21.6 mm
- net Net-(U51C--INB): track 9.09 -> 7.95 mm
- net /digital to analog v2/TO_5V: track 52.1 -> 51.3 mm
- net +5V: track 380.3 -> 379.5 mm
- net +3V3: track 165.7 -> 165.0 mm
- net /digital to analog v2/DAC_OUTPUT: track 11.0 -> 10.3 mm
- net Net-(U45B-+INA): track 6.75 -> 6.02 mm
- net Net-(U51B-+INA): track 5.76 -> 5.02 mm
- net /analog switching/CAL1: track 12.8 -> 12.1 mm
- net /CAL_PATH_EN: track 73.9 -> 73.2 mm
- net /DAC_SCLK: track 46.9 -> 46.2 mm
- net /analog switching/CAL2: track 12.0 -> 11.3 mm
- net /analog switching/AMP_MEASURE: track 11.3 -> 10.6 mm
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- added copper zone on B.Cu, net GND
