File: pcb/benchpod-analog/vbench-pod.kicad_pcb (KiCad board)
At the start: 4 copper layers, 98.5 x 120.2 mm, 237 parts, among them CN1 KH-FPC1.0-H2.0SMT-24P-QCHF, J10 BNC-KYWE-295-W4-N, J11 DB2ERC-3.81-6P-BK, J8 DB2ERC-3.81-2P-BK, J9 DB2ERC-3.81-2P-BK, K1 G6K-2F-Y DC5, K2 G6K-2F-Y DC5, K3 G6K-2F-Y DC5, K4 G6K-2F-Y DC5, Q1 BCP56, U15 TPS7A2045PDBVR, U16 TLV61046ADBVR, U17 TMCP1A106MTRF, U3 TPS7A2050PDQNR, U30 AP2112K-3.3, U36 MCP33131D-10-E/MS, U37 THS4551IRUNR, U38 ADR4540BRZ-R7, U39 AP2112K-1.8TRG1, U40 OPA810IDBVR, U41 LM27761DSGR, U42 LM7705MM/NOPB, U43 DAC8554IPWR, U44 OPA2365AIDR, U45 OPA2992IDR, U46 AP2112K-3.3, U49 TPS65131RGER, U50 TPS7A1901DRBR, U51 OPA2992IDR, U53 TPL7407LAPWR, U58 TCA9554PWR, U61 24C32, U9 XTR116UA/2K5

Commit message: vias, fixes
Parts:
- moved R81 10.8 mm to (76.9, 32.8)
Routing:
- net /analog to digital v2/AMP_MEASURE_IN: track 25.8 -> 17.5 mm
- net GND: track 164.9 -> 169.4 mm, vias 250 -> 517
- net Net-(U9-IIN): track 6.51 -> 10.4 mm
- net /CAL_PATH_EN: track 73.2 -> 69.8 mm
- net +5V: track 379.5 -> 376.3 mm
- net /AMP_MEAS_EN: track 51.2 -> 49.6 mm
- net Net-(J9-Pin_2): track 31.6 -> 33.0 mm
- net +3V3: track 165.0 -> 164.3 mm
- net /CAL2_EN: track 42.9 -> 42.3 mm
- net -5VA: track 69.6 -> 69.0 mm
- net /CAL1_EN: track 49.9 -> 50.4 mm
Other:
- outline, holes or cut-outs redrawn

Commit message: signal improvements
Routing:
- net +5V: track 376.3 -> 372.2 mm
- net +14V_ANA: track 95.9 -> 96.7 mm
- net 5VA: track 180.7 -> 179.9 mm
- net /CAL2_EN: track 42.3 -> 41.5 mm
- net /CAL1_EN: track 50.4 -> 49.9 mm
- net GND: track 169.4 -> 168.9 mm, vias 517 -> 640

Commit message: signal improvements
Routing:
- net 5VA: track 179.9 -> 177.9 mm
- net AREF_4V096: track 138.4 -> 139.0 mm
- net +3V3A: track 131.5 -> 132.0 mm
- net GND: vias 640 -> 653
