File: pcb/benchpod-analog/vbench-pod.kicad_pcb (KiCad board)
At the start: 4 copper layers, 98.5 x 120.2 mm, 237 parts, among them CN1 KH-FPC1.0-H2.0SMT-24P-QCHF, J10 BNC-KYWE-295-W4-N, J11 DB2ERC-3.81-6P-BK, J8 DB2ERC-3.81-2P-BK, J9 DB2ERC-3.81-2P-BK, K1 G6K-2F-Y DC5, K2 G6K-2F-Y DC5, K3 G6K-2F-Y DC5, K4 G6K-2F-Y DC5, Q1 BCP56, U15 TPS7A2045PDBVR, U16 TLV61046ADBVR, U17 TMCP1A106MTRF, U3 TPS7A2050PDQNR, U30 AP2112K-3.3, U36 MCP33131D-10-E/MS, U37 THS4551IRUNR, U38 ADR4540BRZ-R7, U39 AP2112K-1.8TRG1, U40 OPA810IDBVR, U41 LM27761DSGR, U42 LM7705MM/NOPB, U43 DAC8554IPWR, U44 OPA2365AIDR, U45 OPA2992IDR, U46 AP2112K-3.3, U49 TPS65131RGER, U50 TPS7A1901DRBR, U51 OPA2992IDR, U53 TPL7407LAPWR, U58 TCA9554PWR, U61 24C32, U9 XTR116UA/2K5

Commit message: analog module: use reserved JLC stock for C207/C208 and U42
C207/C208 5.1 pF: C2297586 (11 left at JLC) -> C20617868 (FH 0603 C0G 50 V,
100 reserved); op-amp feedback caps, 50 V is plenty. C140 9.1 pF 250 V stays.
U42 LM7705MM/NOPB C129980 -> LM7705MMX/NOPB C2070761 (same chip and
VSSOP-8 package, larger reel; 10 reserved). Schematic and board fields both.

Co-Authored-By: Claude Opus 5.5 <noreply@anthropic.com>
Parts:
- U42: value LM7705MM/NOPB -> LM7705MMX/NOPB
Changed lines of the file:
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@@
 			)
 		)
-		(property "Value" "LM7705MM/NOPB"
+		(property "Value" "LM7705MMX/NOPB"
 			(at 0 6.146 0)
 			(layer "F.Fab")
@@
 			)
 		)
-		(property "LCSC Part" "C129980"
+		(property "LCSC Part" "C2070761"
 			(at 0 0 0)
 			(layer "F.Fab")
@@
 			)
 		)
-		(property "MPN" "LM7705MM/NOPB"
+		(property "MPN" "LM7705MMX/NOPB"
 			(at 0 0 0)
 			(unlocked yes)
@@
 			)
 		)
-		(property "LCSC" "C129980"
+		(property "LCSC" "C2070761"
 			(at 0 0 0)
 			(unlocked yes)
@@
 			)
 		)
-		(property "LCSC" "C2297586"
+		(property "LCSC" "C20617868"
 			(at 0 0 270)
 			(unlocked yes)
@@
 			)
 		)
-		(property "LCSC" "C2297586"
+		(property "LCSC" "C20617868"
 			(at 0 0 0)
 			(unlocked yes)
