File: pcb/benchpod-analog/vbench-pod.kicad_sch (KiCad schematic)
At the start: 7 parts, among them CN1 KH-FPC1.0-H2.0SMT-24P-QCHF, U61 24C32

Commit message: analog module: ÷2 ADC low range (K5)
A second input range for small signals: ±5.46 V (÷2, 167 uV/count)
next to today's ±32.8 V (÷12), 6x the resolution on 0-5 V signals and on
the J8 current input (both share the divider).

- K5 (G6K-2F-Y DC5, same part as K3) driven by U53 OUT5 from U58 P5
  (R185 4.7k pull-down), LOW_RANGE_EN through the root sheet.
- Pole 1 swaps the bottom leg: R91 82.5k + C72 to GND (NC1, off) or
  R182 910k 0.1 % 25 ppm + C269 47 pF to GND (NO1, on). R90 stays in
  series, so 30 V into the D22 clamp is still ~33 uA.
- Pole 2 moves C271 (47 pF 100 V): to GND on the normal range (part of
  the bottom leg; C72 100 -> 51 pF keeps it at ~105 pF with strays), across
  R90 on the low range (top leg 56.4 pF). The open contacts never bridge
  the divider, so the normal range keeps the v3r3 compensation.
- C270 DNP pad for the first-article trim (adc_comp_sweep.py on both
  ranges); R183/R184 0 ohm DNP give the ÷12 divider without K5.
- ADC sheet A3 (like the power and DAC sheets) for room.

Netlist checked against the design; ERC adds only pin_to_pin notes from
the relay symbol's unspecified pin types (as K3/K4). PCB not updated.

Co-Authored-By: Claude Opus 5.5 <noreply@anthropic.com>
Other:
- sheet analog switching ports: added LOW_RANGE_EN; removed none
- sheet analog to digital v2 ports: added LOW_RANGE_EN; removed none
Changed lines of the file:
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@@
+			)
+		)
+		(pin "LOW_RANGE_EN" input
+			(at 171.45 113.03 0)
+			(effects
+				(font
+					(size 1.27 1.27)
+				)
+				(justify right)
 			)
 		)
@@
 			)
 		)
+		(pin "LOW_RANGE_EN" input
+			(at 137.16 93.98 0)
+			(effects
+				(font
+					(size 1.27 1.27)
+				)
+				(justify right)
+			)
+		)
 		(pin "CAL_PATH_EN" input
 			(at 137.16 91.44 0)
@@
 		)
 	)
+	(label "LOW_RANGE_EN"
+		(at 171.45 113.03 0)
+		(effects
+			(font
+				(size 1.27 1.27)
+			)
+			(justify left bottom)
+		)
+	)
+	(label "LOW_RANGE_EN"
+		(at 137.16 93.98 0)
+		(effects
+			(font
+				(size 1.27 1.27)
+			)
+			(justify left bottom)
+		)
+	)
