File: pcb/benchpod-analog/analog-power-v2.kicad_sch (KiCad schematic)
At the start: 103 parts, among them U15 TPS7A2045PDBVR, U16 TLV61046ADBVR, U3 TPS7A2050PDQNR, U38 ADR4540BRZ-R7, U39 AP2112K-1.8TRG1, U41 LM27761DSGR, U42 LM7705MM/NOPB, U46 AP2112K-3.3, U49 TPS65131RGER, U50 TPS7A1901DRBR

Commit message: analog module: use reserved JLC stock for C207/C208 and U42
C207/C208 5.1 pF: C2297586 (11 left at JLC) -> C20617868 (FH 0603 C0G 50 V,
100 reserved); op-amp feedback caps, 50 V is plenty. C140 9.1 pF 250 V stays.
U42 LM7705MM/NOPB C129980 -> LM7705MMX/NOPB C2070761 (same chip and
VSSOP-8 package, larger reel; 10 reserved). Schematic and board fields both.

Co-Authored-By: Claude Opus 5.5 <noreply@anthropic.com>
Parts:
- U42: value LM7705MM/NOPB -> LM7705MMX/NOPB; LCSC C129980 -> C2070761; LCSC Part C129980 -> C2070761; MPN LM7705MM/NOPB -> LM7705MMX/NOPB
Changed lines of the file:
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@@
 			)
 		)
-		(property "Value" "LM7705MM/NOPB"
+		(property "Value" "LM7705MMX/NOPB"
 			(at 327.66 200.66 0)
 			(show_name no)
@@
 			)
 		)
-		(property "MPN" "LM7705MM/NOPB"
+		(property "MPN" "LM7705MMX/NOPB"
 			(at 327.66 233.68 0)
 			(hide yes)
@@
 			)
 		)
-		(property "LCSC Part" "C129980"
+		(property "LCSC Part" "C2070761"
 			(at 327.66 236.22 0)
 			(hide yes)
@@
 			)
 		)
-		(property "LCSC" "C129980"
+		(property "LCSC" "C2070761"
 			(at 327.66 212.09 0)
 			(hide yes)
