File: pcb/benchpod-analog/analog-switching.kicad_sch (KiCad schematic)
At the start: 11 parts, among them U53 TPL7407LAPWR, U58 TCA9554PWR

Commit message: analog module: ÷2 ADC low range (K5)
A second input range for small signals: ±5.46 V (÷2, 167 uV/count)
next to today's ±32.8 V (÷12), 6x the resolution on 0-5 V signals and on
the J8 current input (both share the divider).

- K5 (G6K-2F-Y DC5, same part as K3) driven by U53 OUT5 from U58 P5
  (R185 4.7k pull-down), LOW_RANGE_EN through the root sheet.
- Pole 1 swaps the bottom leg: R91 82.5k + C72 to GND (NC1, off) or
  R182 910k 0.1 % 25 ppm + C269 47 pF to GND (NO1, on). R90 stays in
  series, so 30 V into the D22 clamp is still ~33 uA.
- Pole 2 moves C271 (47 pF 100 V): to GND on the normal range (part of
  the bottom leg; C72 100 -> 51 pF keeps it at ~105 pF with strays), across
  R90 on the low range (top leg 56.4 pF). The open contacts never bridge
  the divider, so the normal range keeps the v3r3 compensation.
- C270 DNP pad for the first-article trim (adc_comp_sweep.py on both
  ranges); R183/R184 0 ohm DNP give the ÷12 divider without K5.
- ADC sheet A3 (like the power and DAC sheets) for room.

Netlist checked against the design; ERC adds only pin_to_pin notes from
the relay symbol's unspecified pin types (as K3/K4). PCB not updated.

Co-Authored-By: Claude Opus 5.5 <noreply@anthropic.com>
Parts:
- added R185: 4.7k, Resistor_SMD:R_0402_1005Metric, symbol Device:R
Connections:
- net GND: now also R185.2; no longer U53.5 (IN5)
- net LOW_RANGE: now reaches U58.10 (P5)
- net LOW_RANGE: now also U53.5 (IN5), R185.1
- net LOW_RANGE_EN: now reaches U53.12 (OUT5)
- no-connect marks 6 -> 4
